File: 07_Schémas/manette_2019/manette_2019.sch (KiCad schematic (older format))
At the start: 7 parts

Commit message: schéma
Parts:
- added JS? (x2): Joystick_RSF_2-Axis, symbol Manette_arcade:Joystick_RSF_2-Axis
- added RV? (x2): R_POT, symbol Device:R_POT
- added SW? (x6): SW_Push, symbol Switch:SW_Push
- added SW?: SW_DPDT_x2, symbol Switch:SW_DPDT_x2
Changed lines of the file:
@@
+	1    0    0    -1
+$EndComp
+$Comp
+L Manette_arcade:Joystick_RSF_2-Axis JS?
+U 1 1 5C7D4903
+P 8850 1300
+F 0 "JS?" H 8270 1403 60  0000 R CNN
+F 1 "Joystick_RSF_2-Axis" H 8270 1297 60  0000 R CNN
+F 2 "" H 8650 1300 60  0001 C CNN
+F 3 "" H 8650 1300 60  0001 C CNN
+	1    8850 1300
+	1    0    0    -1
+$EndComp
+$Comp
+L Manette_arcade:Joystick_RSF_2-Axis JS?
+U 1 1 5C7D49EC
+P 8900 3350
+F 0 "JS?" H 8320 3453 60  0000 R CNN
+F 1 "Joystick_RSF_2-Axis" H 8320 3347 60  0000 R CNN
+F 2 "" H 8700 3350 60  0001 C CNN
+F 3 "" H 8700 3350 60  0001 C CNN
+	1    8900 3350
+	1    0    0    -1
+$EndComp
+$Comp
+L Device:R_POT RV?
+U 1 1 5C7D4ACF
+P 7700 4550
+F 0 "RV?" H 7630 4596 50  0000 R CNN
+F 1 "R_POT" H 7630 4505 50  0000 R CNN
+F 2 "" H 7700 4550 50  0001 C CNN
+F 3 "~" H 7700 4550 50  0001 C CNN
+	1    7700 4550
+	1    0    0    -1
+$EndComp
+$Comp
+L Device:R_POT RV?
+U 1 1 5C7D4B89
+P 7800 5300
+F 0 "RV?" H 7730 5346 50  0000 R CNN
+F 1 "R_POT" H 7730 5255 50  0000 R CNN
+F 2 "" H 7800 5300 50  0001 C CNN
+F 3 "~" H 7800 5300 50  0001 C CNN
+	1    7800 5300
+	1    0    0    -1
+$EndComp
+$Comp
+L Switch:SW_Push SW?
+U 1 1 5C7D4D3A
+P 6200 5350
+F 0 "SW?" H 6200 5635 50  0000 C CNN
+F 1 "SW_Push" H 6200 5544 50  0000 C CNN
+F 2 "" H 6200 5550 50  0001 C CNN
+F 3 "" H 6200 5550 50  0001 C CNN
+	1    6200 5350
+	1    0    0    -1
+$EndComp
+$Comp
+L Switch:SW_Push SW?
+U 1 1 5C7D4D41
+P 6200 5900
+F 0 "SW?" H 6200 6185 50  0000 C CNN
+F 1 "SW_Push" H 6200 6094 50  0000 C CNN
+F 2 "" H 6200 6100 50  0001 C CNN
+F 3 "" H 6200 6100 50  0001 C CNN
+	1    6200 5900
+	1    0    0    -1
+$EndComp
+$Comp
+L Switch:SW_Push SW?
+U 1 1 5C7D4D48
+P 6200 6450
+F 0 "SW?" H 6200 6735 50  0000 C CNN
+F 1 "SW_Push" H 6200 6644 50  0000 C CNN
+F 2 "" H 6200 6650 50  0001 C CNN
+F 3 "" H 6200 6650 50  0001 C CNN
+	1    6200 6450
+	1    0    0    -1
+$EndComp
+$Comp
+L Switch:SW_Push SW?
+U 1 1 5C7D4D4F
+P 6200 7000
+F 0 "SW?" H 6200 7285 50  0000 C CNN
+F 1 "SW_Push" H 6200 7194 50  0000 C CNN
+F 2 "" H 6200 7200 50  0001 C CNN
+F 3 "" H 6200 7200 50  0001 C CNN
+	1    6200 7000
+	1    0    0    -1
+$EndComp
+$Comp
+L Switch:SW_Push SW?
+U 1 1 5C7D4F76
+P 6200 1000
+F 0 "SW?" H 6200 1285 50  0000 C CNN
+F 1 "SW_Push" H 6200 1194 50  0000 C CNN
+F 2 "" H 6200 1200 50  0001 C CNN
+F 3 "" H 6200 1200 50  0001 C CNN
+	1    6200 1000
+	1    0    0    -1
+$EndComp
+$Comp
+L Switch:SW_Push SW?
+U 1 1 5C7D4F7D
+P 6200 1550
+F 0 "SW?" H 6200 1835 50  0000 C CNN
+F 1 "SW_Push" H 6200 1744 50  0000 C CNN
+F 2 "" H 6200 1750 50  0001 C CNN
+F 3 "" H 6200 1750 50  0001 C CNN
+	1    6200 1550
+	1    0    0    -1
+$EndComp
+$Comp
+L Switch:SW_DPDT_x2 SW?
+U 1 1 5C7D5504
+P 4600 5300
+F 0 "SW?" H 4600 5585 50  0000 C CNN
+F 1 "SW_DPDT_x2" H 4600 5494 50  0000 C CNN
+F 2 "" H 4600 5300 50  0001 C CNN
+F 3 "" H 4600 5300 50  0001 C CNN
+	1    4600 5300
 	1    0    0    -1
 $EndComp

Commit message: schéma
Parts:
- added LS?: Speaker, symbol Device:Speaker
Changed lines of the file:
@@
+	1    0    0    -1
+$EndComp
+$Comp
+L Device:Speaker LS?
+U 1 1 5C7D5866
+P 4250 6000
+F 0 "LS?" H 4420 5996 50  0000 L CNN
+F 1 "Speaker" H 4420 5905 50  0000 L CNN
+F 2 "" H 4250 5800 50  0001 C CNN
+F 3 "~" H 4240 5950 50  0001 C CNN
+	1    4250 6000
 	1    0    0    -1
 $EndComp

Commit message: schéma
Parts:
- added J?: Conn_01x10, symbol Connector_Generic:Conn_01x10
- added SW? (x2): SW_Push, symbol Switch:SW_Push
Connections:
- net labels added: +5V, D/C, GND, LCD, MISO, MOSI, RESET, SCK, SD
- wire segments 0 -> 11
Changed lines of the file:
@@
 EESchema Schematic File Version 4
+LIBS:manette_2019-cache
 EELAYER 26 0
 EELAYER END
@@
 	1    0    0    -1
 $EndComp
+Text GLabel 9600 4500 0    50   Input ~ 0
++5V
+Text GLabel 9350 4600 0    50   Output ~ 0
+MISO
+Text GLabel 9600 4700 0    50   Input ~ 0
+SCK
+Text GLabel 9350 4800 0    50   Input ~ 0
+MOSI
+Text GLabel 9550 4900 0    50   UnSpc ~ 0
+LCD
+Text GLabel 9300 5000 0    50   UnSpc ~ 0
+SD
+Text GLabel 9550 5100 0    50   UnSpc ~ 0
+D/C
+Text GLabel 9300 5200 0    50   Input ~ 0
+RESET
+Text GLabel 9550 5300 0    50   Input ~ 0
++5V
+$Comp
+L power:GND #PWR?
+U 1 1 5C7E33B4
+P 9600 5500
+F 0 "#PWR?" H 9600 5250 50  0001 C CNN
+F 1 "GND" H 9605 5327 50  0000 C CNN
+F 2 "" H 9600 5500 50  0001 C CNN
+F 3 "" H 9600 5500 50  0001 C CNN
+	1    9600 5500
+	1    0    0    -1
+$EndComp
+Wire Wire Line
+	9600 5500 9600 5400
+Wire Wire Line
+	9600 5400 9750 5400
+Wire Wire Line
+	9550 5300 9750 5300
+Wire Wire Line
+	9300 5200 9750 5200
+Wire Wire Line
+	9550 5100 9750 5100
+Wire Wire Line
+	9750 5000 9300 5000
+Wire Wire Line
+	9550 4900 9750 4900
+Wire Wire Line
+	9350 4800 9750 4800
+Wire Wire Line
+	9750 4700 9600 4700
+Wire Wire Line
+	9350 4600 9750 4600
+Wire Wire Line
+	9600 4500 9750 4500
+$Comp
+L Connector_Generic:Conn_01x10 J?
+U 1 1 5C7E2DEA
+P 9950 4900
+F 0 "J?" H 10030 4892 50  0000 L CNN
+F 1 "Conn_01x10" H 10030 4801 50  0000 L CNN
+F 2 "" H 9950 4900 50  0001 C CNN
+F 3 "~" H 9950 4900 50  0001 C CNN
+	1    9950 4900
+	1    0    0    -1
+$EndComp
+$Comp
+L Switch:SW_Push SW?
+U 1 1 5C7E3FD7
+P 5450 1000
+F 0 "SW?" H 5450 1285 50  0000 C CNN
+F 1 "SW_Push" H 5450 1194 50  0000 C CNN
+F 2 "" H 5450 1200 50  0001 C CNN
+F 3 "" H 5450 1200 50  0001 C CNN
+	1    5450 1000
+	1    0    0    -1
+$EndComp
+$Comp
+L Switch:SW_Push SW?
+U 1 1 5C7E3FDE
+P 5450 1550
+F 0 "SW?" H 5450 1835 50  0000 C CNN
+F 1 "SW_Push" H 5450 1744 50  0000 C CNN
+F 2 "" H 5450 1750 50  0001 C CNN
+F 3 "" H 5450 1750 50  0001 C CNN
+	1    5450 1550
+	1    0    0    -1
+$EndComp

Commit message: update schéma
Parts:
- added U?: MCP23017, symbol MCP23017:MCP23017
Changed lines of the file:
@@
 L MCU_Module:Arduino_UNO_R3 A1
 U 1 1 5C7D419E
-P 3550 3100
-F 0 "A1" H 3550 4278 50  0000 C CNN
-F 1 "Arduino_UNO_R3" H 3550 4187 50  0000 C CNN
-F 2 "Module:Arduino_UNO_R3" H 3700 2050 50  0001 L CNN
-F 3 "https://www.arduino.cc/en/Main/arduinoBoardUno" H 3350 4150 50  0001 C CNN
-	1    3550 3100
+P 2000 2150
+F 0 "A1" H 2000 3328 50  0000 C CNN
+F 1 "Arduino_UNO_R3" H 2000 3237 50  0000 C CNN
+F 2 "Module:Arduino_UNO_R3" H 2150 1100 50  0001 L CNN
+F 3 "https://www.arduino.cc/en/Main/arduinoBoardUno" H 1800 3200 50  0001 C CNN
+	1    2000 2150
 	1    0    0    -1
 $EndComp
@@
 	1    0    0    -1
 $EndComp
-Text GLabel 9600 4500 0    50   Input ~ 0
+Text GLabel 1450 4350 0    50   Input ~ 0
 +5V
-Text GLabel 9350 4600 0    50   Output ~ 0
+Text GLabel 1200 4450 0    50   Output ~ 0
 MISO
-Text GLabel 9600 4700 0    50   Input ~ 0
+Text GLabel 1450 4550 0    50   Input ~ 0
 SCK
-Text GLabel 9350 4800 0    50   Input ~ 0
+Text GLabel 1200 4650 0    50   Input ~ 0
 MOSI
-Text GLabel 9550 4900 0    50   UnSpc ~ 0
+Text GLabel 1400 4750 0    50   UnSpc ~ 0
 LCD
-Text GLabel 9300 5000 0    50   UnSpc ~ 0
+Text GLabel 1150 4850 0    50   UnSpc ~ 0
 SD
-Text GLabel 9550 5100 0    50   UnSpc ~ 0
+Text GLabel 1400 4950 0    50   UnSpc ~ 0
 D/C
-Text GLabel 9300 5200 0    50   Input ~ 0
+Text GLabel 1150 5050 0    50   Input ~ 0
 RESET
-Text GLabel 9550 5300 0    50   Input ~ 0
+Text GLabel 1400 5150 0    50   Input ~ 0
 +5V
 $Comp
 L power:GND #PWR?
 U 1 1 5C7E33B4
-P 9600 5500
-F 0 "#PWR?" H 9600 5250 50  0001 C CNN
-F 1 "GND" H 9605 5327 50  0000 C CNN
-F 2 "" H 9600 5500 50  0001 C CNN
-F 3 "" H 9600 5500 50  0001 C CNN
-	1    9600 5500
-	1    0    0    -1
-$EndComp
-Wire Wire Line
-	9600 5500 9600 5400
-Wire Wire Line
-	9600 5400 9750 5400
-Wire Wire Line
-	9550 5300 9750 5300
-Wire Wire Line
-	9300 5200 9750 5200
-Wire Wire Line
-	9550 5100 9750 5100
-Wire Wire Line
-	9750 5000 9300 5000
-Wire Wire Line
-	9550 4900 9750 4900
-Wire Wire Line
-	9350 4800 9750 4800
-Wire Wire Line
-	9750 4700 9600 4700
-Wire Wire Line
-	9350 4600 9750 4600
-Wire Wire Line
-	9600 4500 9750 4500
+P 1450 5350
+F 0 "#PWR?" H 1450 5100 50  0001 C CNN
+F 1 "GND" H 1455 5177 50  0000 C CNN
+F 2 "" H 1450 5350 50  0001 C CNN
+F 3 "" H 1450 5350 50  0001 C CNN
+	1    1450 5350
+	1    0    0    -1
+$EndComp
+Wire Wire Line
+	1450 5350 1450 5250
+Wire Wire Line
+	1450 5250 1600 5250
+Wire Wire Line
+	1400 5150 1600 5150
+Wire Wire Line
+	1150 5050 1600 5050
+Wire Wire Line
+	1400 4950 1600 4950
+Wire Wire Line
+	1600 4850 1150 4850
+Wire Wire Line
+	1400 4750 1600 4750
+Wire Wire Line
+	1200 4650 1600 4650
+Wire Wire Line
+	1600 4550 1450 4550
+Wire Wire Line
+	1200 4450 1600 4450
+Wire Wire Line
+	1450 4350 1600 4350
 $Comp
 L Connector_Generic:Conn_01x10 J?
 U 1 1 5C7E2DEA
-P 9950 4900
-F 0 "J?" H 10030 4892 50  0000 L CNN
-F 1 "Conn_01x10" H 10030 4801 50  0000 L CNN
-F 2 "" H 9950 4900 50  0001 C CNN
-F 3 "~" H 9950 4900 50  0001 C CNN
-	1    9950 4900
+P 1800 4750
+F 0 "J?" H 1880 4742 50  0000 L CNN
+F 1 "Conn_01x10" H 1880 4651 50  0000 L CNN
+F 2 "" H 1800 4750 50  0001 C CNN
+F 3 "~" H 1800 4750 50  0001 C CNN
+	1    1800 4750
 	1    0    0    -1
 $EndComp
@@
 	1    0    0    -1
 $EndComp
+$Comp
+L MCP23017:MCP23017 U?
+U 1 1 5C80D464
+P 4150 1900
+F 0 "U?" H 4250 1915 50  0000 C CNN
+F 1 "MCP23017" H 4250 1824 50  0000 C CNN
+F 2 "" H 4250 1850 50  0001 C CNN
+F 3 "" H 4250 1850 50  0001 C CNN
+	1    4150 1900
+	1    0    0    -1
+$EndComp
+Text GLabel 1250 3450 0    50   Input ~ 0
+MISO
+Text GLabel 1250 3750 0    50   Output ~ 0
+SCK
+Text GLabel 2000 3750 0    50   Output ~ 0
+MOSI
+Text GLabel 1800 3550 0    50   UnSpc ~ 0
+LCD
+Text GLabel 2200 3600 0    50   UnSpc ~ 0
+SD
+Text GLabel 2350 3800 0    50   UnSpc ~ 0
+D/C
+Text GLabel 2550 3500 0    50   Output ~ 0
+RESET
 $EndSCHEMATC

Commit message: schéma update
Parts:
- removed A1: Arduino_UNO_R3, Module:Arduino_UNO_R3, symbol MCU_Module:Arduino_UNO_R3
- added U?: ATmega328-PU, Package_DIP:DIP-28_W7.62mm, symbol MCU_Microchip_ATmega:ATmega328-PU
Connections:
- net labels added: Left_joystick_analog_x, Left_joystick_analog_y, Left_joystick_button, Left_trigger, Right_joystick_analog_x, Right_joystick_analog_y, Right_joystick_button, Right_trigger, SCL, SDA
- wire segments 11 -> 21

Commit message: update schéma
Parts:
- removed SW? (x2): SW_Push, symbol Switch:SW_Push
- added D?: LED, symbol Device:LED
- added R?: R, symbol Device:R
- added U?: ULN2803A, symbol Transistor_Array:ULN2803A
- added Y?: Resonator, symbol Device:Resonator
- SW1: renamed from SW?; value SW_Push -> Button_A
- SW?: value SW_Push -> Button_X
- SW?: value SW_Push -> Button_Y
- SW?: value SW_Push -> Button_Start
- SW?: value SW_Push -> Button_Select
- SW?: value SW_Push -> Button_Gauche
- SW?: value SW_Push -> Button_Bas
- SW?: value SW_Push -> Button_B
- SW?: value SW_Push -> Button_Droite
- SW?: value SW_Push -> Button_Haut
Connections:
- net labels added: L_joystick_analog_x, L_joystick_analog_y, L_joystick_button, L_trigger, R_joystick_analog_x, R_joystick_analog_y, R_joystick_button, R_trigger
- wire segments 21 -> 31
Changed lines of the file:
@@
 P 6200 2100
 F 0 "SW?" H 6200 2385 50  0000 C CNN
-F 1 "SW_Push" H 6200 2294 50  0000 C CNN
+F 1 "Button_X" H 6200 2294 50  0000 C CNN
 F 2 "" H 6200 2300 50  0001 C CNN
 F 3 "" H 6200 2300 50  0001 C CNN
@@
 P 6200 2650
 F 0 "SW?" H 6200 2935 50  0000 C CNN
-F 1 "SW_Push" H 6200 2844 50  0000 C CNN
+F 1 "Button_Y" H 6200 2844 50  0000 C CNN
 F 2 "" H 6200 2850 50  0001 C CNN
 F 3 "" H 6200 2850 50  0001 C CNN
@@
 P 6200 3150
 F 0 "SW?" H 6200 3435 50  0000 C CNN
-F 1 "SW_Push" H 6200 3344 50  0000 C CNN
+F 1 "Button_Start" H 6200 3344 50  0000 C CNN
 F 2 "" H 6200 3350 50  0001 C CNN
 F 3 "" H 6200 3350 50  0001 C CNN
@@
 P 6200 3700
 F 0 "SW?" H 6200 3985 50  0000 C CNN
-F 1 "SW_Push" H 6200 3894 50  0000 C CNN
+F 1 "Button_Select" H 6200 3894 50  0000 C CNN
 F 2 "" H 6200 3900 50  0001 C CNN
 F 3 "" H 6200 3900 50  0001 C CNN
 	1    6200 3700
-	1    0    0    -1
-$EndComp
-$Comp
-L Switch:SW_Push SW?
-U 1 1 5C7D46B3
-P 6200 4250
-F 0 "SW?" H 6200 4535 50  0000 C CNN
-F 1 "SW_Push" H 6200 4444 50  0000 C CNN
-F 2 "" H 6200 4450 50  0001 C CNN
-F 3 "" H 6200 4450 50  0001 C CNN
-	1    6200 4250
-	1    0    0    -1
-$EndComp
-$Comp
-L Switch:SW_Push SW?
-U 1 1 5C7D46BA
-P 6800 4250
-F 0 "SW?" H 6800 4535 50  0000 C CNN
-F 1 "SW_Push" H 6800 4444 50  0000 C CNN
-F 2 "" H 6800 4450 50  0001 C CNN
-F 3 "" H 6800 4450 50  0001 C CNN
-	1    6800 4250
 	1    0    0    -1
 $EndComp
@@
 $Comp
 L Switch:SW_Push SW?
-U 1 1 5C7D4D41
-P 6800 3700
-F 0 "SW?" H 6800 3985 50  0000 C CNN
-F 1 "SW_Push" H 6800 3894 50  0000 C CNN
-F 2 "" H 6800 3900 50  0001 C CNN
-F 3 "" H 6800 3900 50  0001 C CNN
-	1    6800 3700
-	1    0    0    -1
-$EndComp
-$Comp
-L Switch:SW_Push SW?
 U 1 1 5C7D4D48
 P 6800 2100
 F 0 "SW?" H 6800 2385 50  0000 C CNN
-F 1 "SW_Push" H 6800 2294 50  0000 C CNN
+F 1 "Button_Gauche" H 6800 2294 50  0000 C CNN
 F 2 "" H 6800 2300 50  0001 C CNN
 F 3 "" H 6800 2300 50  0001 C CNN
@@
 P 6800 2650
 F 0 "SW?" H 6800 2935 50  0000 C CNN
-F 1 "SW_Push" H 6800 2844 50  0000 C CNN
+F 1 "Button_Bas" H 6800 2844 50  0000 C CNN
 F 2 "" H 6800 2850 50  0001 C CNN
 F 3 "" H 6800 2850 50  0001 C CNN
@@
 $EndComp
 $Comp
-L Switch:SW_Push SW?
+L Switch:SW_Push SW1
 U 1 1 5C7D4F76
 P 6200 1000
-F 0 "SW?" H 6200 1285 50  0000 C CNN
-F 1 "SW_Push" H 6200 1194 50  0000 C CNN
+F 0 "SW1" H 6200 1285 50  0000 C CNN
+F 1 "Button_A" H 6200 1194 50  0000 C CNN
 F 2 "" H 6200 1200 50  0001 C CNN
 F 3 "" H 6200 1200 50  0001 C CNN
@@
 P 6200 1550
 F 0 "SW?" H 6200 1835 50  0000 C CNN
-F 1 "SW_Push" H 6200 1744 50  0000 C CNN
+F 1 "Button_B" H 6200 1744 50  0000 C CNN
 F 2 "" H 6200 1750 50  0001 C CNN
 F 3 "" H 6200 1750 50  0001 C CNN
@@
 L Switch:SW_DPDT_x2 SW?
 U 1 1 5C7D5504
-P 7050 4950
-F 0 "SW?" H 7050 5235 50  0000 C CNN
-F 1 "SW_DPDT_x2" H 7050 5144 50  0000 C CNN
-F 2 "" H 7050 4950 50  0001 C CNN
-F 3 "" H 7050 4950 50  0001 C CNN
-	1    7050 4950
+P 6900 4250
+F 0 "SW?" H 6900 4535 50  0000 C CNN
+F 1 "SW_DPDT_x2" H 6900 4444 50  0000 C CNN
+F 2 "" H 6900 4250 50  0001 C CNN
+F 3 "" H 6900 4250 50  0001 C CNN
+	1    6900 4250
 	1    0    0    -1
 $EndComp
@@
 L Device:Speaker LS?
 U 1 1 5C7D5866
-P 7050 5600
-F 0 "LS?" H 7220 5596 50  0000 L CNN
-F 1 "Speaker" H 7220 5505 50  0000 L CNN
-F 2 "" H 7050 5400 50  0001 C CNN
-F 3 "~" H 7040 5550 50  0001 C CNN
-	1    7050 5600
+P 5600 4750
+F 0 "LS?" H 5770 4746 50  0000 L CNN
+F 1 "Speaker" H 5770 4655 50  0000 L CNN
+F 2 "" H 5600 4550 50  0001 C CNN
+F 3 "~" H 5590 4700 50  0001 C CNN
+	1    5600 4750
 	1    0    0    -1
 $EndComp
@@
 P 6800 1000
 F 0 "SW?" H 6800 1285 50  0000 C CNN
-F 1 "SW_Push" H 6800 1194 50  0000 C CNN
+F 1 "Button_Droite" H 6800 1194 50  0000 C CNN
 F 2 "" H 6800 1200 50  0001 C CNN
 F 3 "" H 6800 1200 50  0001 C CNN
@@
 P 6800 1550
 F 0 "SW?" H 6800 1835 50  0000 C CNN
-F 1 "SW_Push" H 6800 1744 50  0000 C CNN
+F 1 "Button_Haut" H 6800 1744 50  0000 C CNN
 F 2 "" H 6800 1750 50  0001 C CNN
 F 3 "" H 6800 1750 50  0001 C CNN
@@
 L MCP23017:MCP23017 U?
 U 1 1 5C80D464
-P 4250 1450
-F 0 "U?" H 4350 1465 50  0000 C CNN
-F 1 "MCP23017" H 4350 1374 50  0000 C CNN
-F 2 "" H 4350 1400 50  0001 C CNN
-F 3 "" H 4350 1400 50  0001 C CNN
-	1    4250 1450
+P 4100 1450
+F 0 "U?" H 4200 1465 50  0000 C CNN
+F 1 "MCP23017" H 4200 1374 50  0000 C CNN
+F 2 "" H 4200 1400 50  0001 C CNN
+F 3 "" H 4200 1400 50  0001 C CNN
+	1    4100 1450
 	1    0    0    -1
 $EndComp
@@
 Text GLabel 2450 2650 2    50   Output ~ 0
 SCL
-Text GLabel 3800 3400 0    50   Input ~ 0
+Text GLabel 3650 3400 0    50   Input ~ 0
 SCL
-Text GLabel 3800 3550 0    50   Input ~ 0
+Text GLabel 3650 3550 0    50   Input ~ 0
 SDA
 $Comp
@@
 L power:GND #PWR?
 U 1 1 5C816DC7
-P 3650 3100
-F 0 "#PWR?" H 3650 2850 50  0001 C CNN
-F 1 "GND" H 3655 2927 50  0000 C CNN
-F 2 "" H 3650 3100 50  0001 C CNN
-F 3 "" H 3650 3100 50  0001 C CNN
-	1    3650 3100
-	1    0    0    -1
-$EndComp
-Wire Wire Line
-	3650 3100 3800 3100
+P 3500 3100
+F 0 "#PWR?" H 3500 2850 50  0001 C CNN
+F 1 "GND" H 3505 2927 50  0000 C CNN
+F 2 "" H 3500 3100 50  0001 C CNN
+F 3 "" H 3500 3100 50  0001 C CNN
+	1    3500 3100
+	1    0    0    -1
+$EndComp
+Wire Wire Line
+	3500 3100 3650 3100
 $Comp
 L power:GND #PWR?
@@
 Text GLabel 9400 3150 1    50   Input ~ 0
 +5V
-Text GLabel 4900 1750 2    50   Input ~ 0
-Right_joystick_analog_x
-Text GLabel 4900 1900 2    50   Input ~ 0
-Right_joystick_analog_y
-Text GLabel 4900 2050 2    50   Input ~ 0
-Right_joystick_button
-Text GLabel 4900 2200 2    50   Input ~ 0
-Left_joystick_analog_x
-Text GLabel 4900 2350 2    50   Input ~ 0
-Left_joystick_analog_y
-Text GLabel 4900 2500 2    50   Input ~ 0
-Left_joystick_button
-Text GLabel 4900 2800 2    50   Output ~ 0
-Left_trigger
-Text GLabel 4900 2650 2    50   Output ~ 0
-Right_trigger
+Text GLabel 4750 1750 2    50   Input ~ 0
+R_joystick_analog_x
+Text GLabel 4750 1900 2    50   Input ~ 0
+R_joystick_analog_y
+Text GLabel 4750 2350 2    50   Input ~ 0
+R_joystick_button
+Text GLabel 4750 2050 2    50   Input ~ 0
+L_joystick_analog_x
+Text GLabel 4750 2200 2    50   Input ~ 0
+L_joystick_analog_y
+Text GLabel 4750 2500 2    50   Input ~ 0
+L_joystick_button
+Text GLabel 4750 2800 2    50   Output ~ 0
+L_trigger
+Text GLabel 4750 2650 2    50   Output ~ 0
+R_trigger
+$Comp
+L Switch:SW_Push SW?
+U 1 1 5C7D4D41
+P 6800 3700
+F 0 "SW?" H 6800 3985 50  0000 C CNN
+F 1 "SW_Push" H 6800 3894 50  0000 C CNN
+F 2 "" H 6800 3900 50  0001 C CNN
+F 3 "" H 6800 3900 50  0001 C CNN
+	1    6800 3700
+	1    0    0    -1
+$EndComp
+$Comp
+L Transistor_Array:ULN2803A U?
+U 1 1 5C82C60F
+P 4350 5150
+F 0 "U?" H 4350 5717 50  0000 C CNN
+F 1 "ULN2803A" H 4350 5626 50  0000 C CNN
+F 2 "" H 4400 4500 50  0001 L CNN
+F 3 "http://www.ti.com/lit/ds/symlink/uln2803a.pdf" H 4450 4950 50  0001 C CNN
+	1    4350 5150
+	1    0    0    -1
+$EndComp
+$Comp
+L Device:Resonator Y?
+U 1 1 5C82CAB8
+P 2900 1900
+F 0 "Y?" V 3200 1850 50  0000 L CNN
+F 1 "Resonator" V 3150 1700 50  0000 L CNN
+F 2 "" H 2875 1900 50  0001 C CNN
+F 3 "~" H 2875 1900 50  0001 C CNN
+	1    2900 1900
+	0    -1   -1   0
+$EndComp
+$Comp
+L power:GND #PWR?
+U 1 1 5C82D22E
+P 3200 2000
+F 0 "#PWR?" H 3200 1750 50  0001 C CNN
+F 1 "GND" H 3205 1827 50  0000 C CNN
+F 2 "" H 3200 2000 50  0001 C CNN
+F 3 "" H 3200 2000 50  0001 C CNN
+	1    3200 2000
+	1    0    0    -1
+$EndComp
+Wire Wire Line
+	3200 2000 3200 1900
+Wire Wire Line
+	3200 1900 3100 1900
+Wire Wire Line
+	2900 2050 2900 2100
+Wire Wire Line
+	2900 2100 2750 2100
+Wire Wire Line
+	2750 2100 2750 1950
+Wire Wire Line
+	2900 1750 2900 1700
+Wire Wire Line
+	2900 1700 2750 1700
+Wire Wire Line
+	2750 1700 2750 1850
+Wire Wire Line
+	2450 1850 2750 1850
+Wire Wire Line
+	2750 1950 2450 1950
+$Comp
+L Device:LED D?
+U 1 1 5C83283C
+P 6750 5600
+F 0 "D?" H 6741 5816 50  0000 C CNN
+F 1 "LED" H 6741 5725 50  0000 C CNN
+F 2 "" H 6750 5600 50  0001 C CNN
+F 3 "~" H 6750 5600 50  0001 C CNN
+	1    6750 5600
+	1    0    0    -1
+$EndComp
+$Comp
+L Device:R R?
+U 1 1 5C8328E9
+P 5950 5800
+F 0 "R?" H 6020 5846 50  0000 L CNN
+F 1 "R" H 6020 5755 50  0000 L CNN
+F 2 "" V 5880 5800 50  0001 C CNN
+F 3 "~" H 5950 5800 50  0001 C CNN
+	1    5950 5800
+	1    0    0    -1
+$EndComp
 $EndSCHEMATC

Commit message: schéma
Parts:
- removed SW?: SW_DPDT_x2, symbol Switch:SW_DPDT_x2
- added SW13: Calib, symbol Manette_arcade:SW_Push
- added SW14: Power On/Off, symbol Switch:SW_DPST_x2
- SW11: renamed from SW?; value SW_Push -> R_button
- SW12: renamed from SW?; value SW_Push -> L_button
- gave numbers to parts that had none: 15
Other:
- moved on the sheet: U1

Commit message: Started schéma pour le test bench, cahier des charges
Parts:
- SW11: value R_button -> R_bumper
- SW12: value L_button -> L_bumper
Changed lines of the file:
@@
 P 6800 3150
 F 0 "SW11" H 6800 3435 50  0000 C CNN
-F 1 "R_button" H 6800 3344 50  0000 C CNN
+F 1 "R_bumper" H 6800 3344 50  0000 C CNN
 F 2 "" H 6800 3350 50  0001 C CNN
 F 3 "" H 6800 3350 50  0001 C CNN
@@
 P 6800 3700
 F 0 "SW12" H 6800 3985 50  0000 C CNN
-F 1 "L_button" H 6800 3894 50  0000 C CNN
+F 1 "L_bumper" H 6800 3894 50  0000 C CNN
 F 2 "" H 6800 3900 50  0001 C CNN
 F 3 "" H 6800 3900 50  0001 C CNN
