File: 07_Schémas/manette_2019/manette_2019.sch (KiCad schematic (older format))
At the start: 26 parts, among them J1 Conn_01x10, SW1 Button_A, SW10 Button_Bas, SW11 R_bumper, SW12 L_bumper, SW13 Calib, SW14 Power On/Off, SW2 Button_B, SW3 Button_X, SW4 Button_Y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

Commit message: Cahier des charges
Connections:
- wire segments 31 -> 40
Changed lines of the file:
@@
 L Device:Speaker LS?
 U 1 1 5C7D5866
-P 6050 4850
-F 0 "LS?" H 6220 4846 50  0000 L CNN
-F 1 "Speaker" H 6220 4755 50  0000 L CNN
-F 2 "" H 6050 4650 50  0001 C CNN
-F 3 "~" H 6040 4800 50  0001 C CNN
-	1    6050 4850
+P 5050 5900
+F 0 "LS?" H 5220 5896 50  0000 L CNN
+F 1 "Speaker" H 5220 5805 50  0000 L CNN
+F 2 "" H 5050 5700 50  0001 C CNN
+F 3 "~" H 5040 5850 50  0001 C CNN
+	1    5050 5900
 	1    0    0    -1
 $EndComp
@@
 L Transistor_Array:ULN2803A U3
 U 1 1 5C82C60F
-P 4350 5150
-F 0 "U3" H 4350 5717 50  0000 C CNN
-F 1 "ULN2803A" H 4350 5626 50  0000 C CNN
-F 2 "" H 4400 4500 50  0001 L CNN
-F 3 "http://www.ti.com/lit/ds/symlink/uln2803a.pdf" H 4450 4950 50  0001 C CNN
-	1    4350 5150
+P 3900 6200
+F 0 "U3" H 3900 6767 50  0000 C CNN
+F 1 "ULN2803A" H 3900 6676 50  0000 C CNN
+F 2 "" H 3950 5550 50  0001 L CNN
+F 3 "http://www.ti.com/lit/ds/symlink/uln2803a.pdf" H 4000 6000 50  0001 C CNN
+	1    3900 6200
 	1    0    0    -1
 $EndComp
@@
 L Device:LED D?
 U 1 1 5C83283C
-P 6600 5400
-F 0 "D?" H 6591 5616 50  0000 C CNN
-F 1 "LED" H 6591 5525 50  0000 C CNN
-F 2 "" H 6600 5400 50  0001 C CNN
-F 3 "~" H 6600 5400 50  0001 C CNN
-	1    6600 5400
+P 5550 6450
+F 0 "D?" H 5541 6666 50  0000 C CNN
+F 1 "LED" H 5541 6575 50  0000 C CNN
+F 2 "" H 5550 6450 50  0001 C CNN
+F 3 "~" H 5550 6450 50  0001 C CNN
+	1    5550 6450
 	1    0    0    -1
 $EndComp
@@
 L Device:R R?
 U 1 1 5C8328E9
-P 6100 5400
-F 0 "R?" H 6170 5446 50  0000 L CNN
-F 1 "R" H 6170 5355 50  0000 L CNN
-F 2 "" V 6030 5400 50  0001 C CNN
-F 3 "~" H 6100 5400 50  0001 C CNN
-	1    6100 5400
+P 5050 6450
+F 0 "R?" H 5120 6496 50  0000 L CNN
+F 1 "R" H 5120 6405 50  0000 L CNN
+F 2 "" V 4980 6450 50  0001 C CNN
+F 3 "~" H 5050 6450 50  0001 C CNN
+	1    5050 6450
 	0    -1   -1   0
 $EndComp
@@
 	1    0    0    -1
 $EndComp
+Wire Wire Line
+	4850 6000 4300 6000
+$Comp
+L power:+5V #PWR?
+U 1 1 5C865522
+P 4700 5650
+F 0 "#PWR?" H 4700 5500 50  0001 C CNN
+F 1 "+5V" H 4715 5823 50  0000 C CNN
+F 2 "" H 4700 5650 50  0001 C CNN
+F 3 "" H 4700 5650 50  0001 C CNN
+	1    4700 5650
+	1    0    0    -1
+$EndComp
+Wire Wire Line
+	4850 5900 4700 5900
+Wire Wire Line
+	4700 5900 4700 5650
+Wire Wire Line
+	4900 6450 4600 6450
+Wire Wire Line
+	4600 6450 4600 6100
+Wire Wire Line
+	4600 6100 4300 6100
+Wire Wire Line
+	5400 6450 5200 6450
+$Comp
+L power:+5V #PWR?
+U 1 1 5C866717
+P 5850 6200
+F 0 "#PWR?" H 5850 6050 50  0001 C CNN
+F 1 "+5V" H 5865 6373 50  0000 C CNN
+F 2 "" H 5850 6200 50  0001 C CNN
+F 3 "" H 5850 6200 50  0001 C CNN
+	1    5850 6200
+	1    0    0    -1
+$EndComp
+Wire Wire Line
+	5850 6450 5850 6200
+Wire Wire Line
+	5700 6450 5850 6450
 $EndSCHEMATC

Commit message: update
Parts:
- added D?: LED, symbol Device:LED
- added D?: D, symbol Device:D
- added R? (x2): R, symbol Device:R
Connections:
- net labels added: Buzzer, Connected, Power
- wire segments 40 -> 52
Changed lines of the file:
@@
 L Device:Speaker LS?
 U 1 1 5C7D5866
-P 5050 5900
-F 0 "LS?" H 5220 5896 50  0000 L CNN
-F 1 "Speaker" H 5220 5805 50  0000 L CNN
-F 2 "" H 5050 5700 50  0001 C CNN
-F 3 "~" H 5040 5850 50  0001 C CNN
-	1    5050 5900
+P 5600 6700
+F 0 "LS?" H 5550 6400 50  0000 L CNN
+F 1 "Speaker" H 5450 6300 50  0000 L CNN
+F 2 "" H 5600 6500 50  0001 C CNN
+F 3 "~" H 5590 6650 50  0001 C CNN
+	1    5600 6700
 	1    0    0    -1
 $EndComp
@@
 L Device:LED D?
 U 1 1 5C83283C
-P 5550 6450
-F 0 "D?" H 5541 6666 50  0000 C CNN
-F 1 "LED" H 5541 6575 50  0000 C CNN
-F 2 "" H 5550 6450 50  0001 C CNN
-F 3 "~" H 5550 6450 50  0001 C CNN
-	1    5550 6450
-	1    0    0    -1
+P 5350 6000
+F 0 "D?" H 5341 6216 50  0000 C CNN
+F 1 "LED" H 5341 6125 50  0000 C CNN
+F 2 "" H 5350 6000 50  0001 C CNN
+F 3 "~" H 5350 6000 50  0001 C CNN
+	1    5350 6000
+	1    0    0    1
 $EndComp
 $Comp
 L Device:R R?
 U 1 1 5C8328E9
-P 5050 6450
-F 0 "R?" H 5120 6496 50  0000 L CNN
-F 1 "R" H 5120 6405 50  0000 L CNN
-F 2 "" V 4980 6450 50  0001 C CNN
-F 3 "~" H 5050 6450 50  0001 C CNN
-	1    5050 6450
-	0    -1   -1   0
+P 4850 6000
+F 0 "R?" H 4920 6046 50  0000 L CNN
+F 1 "R" H 4920 5955 50  0000 L CNN
+F 2 "" V 4780 6000 50  0001 C CNN
+F 3 "~" H 4850 6000 50  0001 C CNN
+	1    4850 6000
+	0    -1   1    0
 $EndComp
 $Comp
@@
 	1    0    0    -1
 $EndComp
-Wire Wire Line
-	4850 6000 4300 6000
-$Comp
-L power:+5V #PWR?
-U 1 1 5C865522
-P 4700 5650
-F 0 "#PWR?" H 4700 5500 50  0001 C CNN
-F 1 "+5V" H 4715 5823 50  0000 C CNN
-F 2 "" H 4700 5650 50  0001 C CNN
-F 3 "" H 4700 5650 50  0001 C CNN
-	1    4700 5650
-	1    0    0    -1
-$EndComp
-Wire Wire Line
-	4850 5900 4700 5900
-Wire Wire Line
-	4700 5900 4700 5650
-Wire Wire Line
-	4900 6450 4600 6450
-Wire Wire Line
-	4600 6450 4600 6100
-Wire Wire Line
-	4600 6100 4300 6100
-Wire Wire Line
-	5400 6450 5200 6450
 $Comp
 L power:+5V #PWR?
 U 1 1 5C866717
-P 5850 6200
-F 0 "#PWR?" H 5850 6050 50  0001 C CNN
-F 1 "+5V" H 5865 6373 50  0000 C CNN
-F 2 "" H 5850 6200 50  0001 C CNN
-F 3 "" H 5850 6200 50  0001 C CNN
-	1    5850 6200
-	1    0    0    -1
-$EndComp
-Wire Wire Line
-	5850 6450 5850 6200
-Wire Wire Line
-	5700 6450 5850 6450
+P 5850 5750
+F 0 "#PWR?" H 5850 5600 50  0001 C CNN
+F 1 "+5V" H 5865 5923 50  0000 C CNN
+F 2 "" H 5850 5750 50  0001 C CNN
+F 3 "" H 5850 5750 50  0001 C CNN
+	1    5850 5750
+	1    0    0    -1
+$EndComp
+Wire Wire Line
+	5850 6000 5850 5750
+$Comp
+L power:GND #PWR?
+U 1 1 5C8638D7
+P 3900 6900
+F 0 "#PWR?" H 3900 6650 50  0001 C CNN
+F 1 "GND" H 3905 6727 50  0000 C CNN
+F 2 "" H 3900 6900 50  0001 C CNN
+F 3 "" H 3900 6900 50  0001 C CNN
+	1    3900 6900
+	1    0    0    -1
+$EndComp
+Text GLabel 3500 6200 0    50   Input ~ 0
+Buzzer
+$Comp
+L Device:R R?
+U 1 1 5C865F77
+P 4850 6700
+F 0 "R?" H 4920 6746 50  0000 L CNN
+F 1 "R" H 4920 6655 50  0000 L CNN
+F 2 "" V 4780 6700 50  0001 C CNN
+F 3 "~" H 4850 6700 50  0001 C CNN
+	1    4850 6700
+	0    -1   -1   0
+$EndComp
+$Comp
+L Device:LED D?
+U 1 1 5C86BA29
+P 5350 6300
+F 0 "D?" H 5341 6516 50  0000 C CNN
+F 1 "LED" H 5341 6425 50  0000 C CNN
+F 2 "" H 5350 6300 50  0001 C CNN
+F 3 "~" H 5350 6300 50  0001 C CNN
+	1    5350 6300
+	1    0    0    1
+$EndComp
+$Comp
+L Device:R R?
+U 1 1 5C86BA30
+P 4850 6300
+F 0 "R?" H 4920 6346 50  0000 L CNN
+F 1 "R" H 4920 6255 50  0000 L CNN
+F 2 "" V 4780 6300 50  0001 C CNN
+F 3 "~" H 4850 6300 50  0001 C CNN
+	1    4850 6300
+	0    -1   1    0
+$EndComp
+Wire Wire Line
+	5200 6300 5000 6300
+Wire Wire Line
+	5200 6000 5000 6000
+Wire Wire Line
+	5850 6300 5850 6000
+Connection ~ 5850 6000
+Wire Wire Line
+	4700 6000 4300 6000
+Wire Wire Line
+	4300 6100 4550 6100
+Wire Wire Line
+	4550 6100 4550 6300
+Wire Wire Line
+	4550 6300 4700 6300
+Wire Wire Line
+	5000 6700 5050 6700
+Wire Wire Line
+	4700 6700 4450 6700
+Wire Wire Line
+	4450 6700 4450 6200
+Wire Wire Line
+	4450 6200 4300 6200
+Wire Wire Line
+	5850 7200 5850 6300
+Connection ~ 5850 6300
+$Comp
+L Device:D D?
+U 1 1 5C878C9C
+P 5050 6850
+F 0 "D?" H 5050 7066 50  0000 C CNN
+F 1 "D" H 5050 6975 50  0000 C CNN
+F 2 "" H 5050 6850 50  0001 C CNN
+F 3 "~" H 5050 6850 50  0001 C CNN
+	1    5050 6850
+	0    -1   -1   0
+$EndComp
+Wire Wire Line
+	5500 6300 5850 6300
+Wire Wire Line
+	5500 6000 5850 6000
+Connection ~ 5050 6700
+Wire Wire Line
+	5050 7200 5050 7000
+Wire Wire Line
+	5050 7200 5250 7200
+Wire Wire Line
+	5250 7200 5250 6800
+Wire Wire Line
+	5250 6800 5400 6800
+Connection ~ 5250 7200
+Wire Wire Line
+	5250 7200 5850 7200
+Wire Wire Line
+	5050 6700 5400 6700
+Text GLabel 3500 6100 0    50   Input ~ 0
+Power
+Text GLabel 3500 6000 0    50   Input ~ 0
+Connected
+Text GLabel 2750 3350 2    50   Output ~ 0
+Connected
+Text GLabel 2750 3250 2    50   Output ~ 0
+Power
+Text GLabel 2750 3150 2    50   Output ~ 0
+Buzzer
 $EndSCHEMATC

Commit message: update schéma
Parts:
- SW10: value Button_Bas -> Button_DOWN
- SW5: value Button_Start -> Button_START
- SW6: value Button_Select -> Button_SELECT
- SW7: value Button_Droite -> Button_RIGHT
- SW8: value Button_Haut -> Button_UP
- SW9: value Button_Gauche -> Button_LEFT
Connections:
- net labels added: Button_A, Button_B, Button_DOWN, Button_LEFT, Button_RIGHT, Button_SELECT, Button_START, Button_UP, Button_X, Button_Y, L_Bumper, R_Bumper
Changed lines of the file:
@@
 P 6200 3150
 F 0 "SW5" H 6200 3435 50  0000 C CNN
-F 1 "Button_Start" H 6200 3344 50  0000 C CNN
+F 1 "Button_START" H 6200 3344 50  0000 C CNN
 F 2 "" H 6200 3350 50  0001 C CNN
 F 3 "" H 6200 3350 50  0001 C CNN
@@
 P 6200 3700
 F 0 "SW6" H 6200 3985 50  0000 C CNN
-F 1 "Button_Select" H 6200 3894 50  0000 C CNN
+F 1 "Button_SELECT" H 6200 3894 50  0000 C CNN
 F 2 "" H 6200 3900 50  0001 C CNN
 F 3 "" H 6200 3900 50  0001 C CNN
@@
 P 6800 2100
 F 0 "SW9" H 6800 2385 50  0000 C CNN
-F 1 "Button_Gauche" H 6800 2294 50  0000 C CNN
+F 1 "Button_LEFT" H 6800 2294 50  0000 C CNN
 F 2 "" H 6800 2300 50  0001 C CNN
 F 3 "" H 6800 2300 50  0001 C CNN
@@
 P 6800 2650
 F 0 "SW10" H 6800 2935 50  0000 C CNN
-F 1 "Button_Bas" H 6800 2844 50  0000 C CNN
+F 1 "Button_DOWN" H 6800 2844 50  0000 C CNN
 F 2 "" H 6800 2850 50  0001 C CNN
 F 3 "" H 6800 2850 50  0001 C CNN
@@
 P 6800 1000
 F 0 "SW7" H 6800 1285 50  0000 C CNN
-F 1 "Button_Droite" H 6800 1194 50  0000 C CNN
+F 1 "Button_RIGHT" H 6800 1194 50  0000 C CNN
 F 2 "" H 6800 1200 50  0001 C CNN
 F 3 "" H 6800 1200 50  0001 C CNN
@@
 P 6800 1550
 F 0 "SW8" H 6800 1835 50  0000 C CNN
-F 1 "Button_Haut" H 6800 1744 50  0000 C CNN
+F 1 "Button_UP" H 6800 1744 50  0000 C CNN
 F 2 "" H 6800 1750 50  0001 C CNN
 F 3 "" H 6800 1750 50  0001 C CNN
@@
 L MCP23017:MCP23017 U2
 U 1 1 5C80D464
-P 4400 1450
-F 0 "U2" H 4500 1465 50  0000 C CNN
-F 1 "MCP23017" H 4500 1374 50  0000 C CNN
-F 2 "" H 4500 1400 50  0001 C CNN
-F 3 "" H 4500 1400 50  0001 C CNN
-	1    4400 1450
-	1    0    0    -1
-$EndComp
-Text GLabel 2750 1650 2    50   Input ~ 0
+P 4350 2850
+F 0 "U2" H 4450 2865 50  0000 C CNN
+F 1 "MCP23017" H 4450 2774 50  0000 C CNN
+F 2 "" H 4450 2800 50  0001 C CNN
+F 3 "" H 4450 2800 50  0001 C CNN
+	1    4350 2850
+	1    0    0    -1
+$EndComp
+Text GLabel 2050 6050 2    50   Input ~ 0
 MISO
-Text GLabel 2750 1750 2    50   Output ~ 0
+Text GLabel 2050 6200 2    50   Output ~ 0
 SCK
-Text GLabel 2750 1550 2    50   Output ~ 0
+Text GLabel 2050 5950 2    50   Output ~ 0
 MOSI
-Text GLabel 2750 1250 2    50   UnSpc ~ 0
+Text GLabel 2050 5650 2    50   UnSpc ~ 0
 LCD
-Text GLabel 2750 3650 2    50   UnSpc ~ 0
+Text GLabel 2050 5500 2    50   UnSpc ~ 0
 SD
-Text GLabel 2750 1350 2    50   UnSpc ~ 0
+Text GLabel 2050 5750 2    50   UnSpc ~ 0
 D/C
-Text GLabel 2750 1450 2    50   Output ~ 0
+Text GLabel 2050 5850 2    50   Output ~ 0
 RESET
 Text GLabel 2750 2550 2    50   Output ~ 0
@@
 Text GLabel 2750 2650 2    50   Output ~ 0
 SCL
-Text GLabel 3950 3400 0    50   Input ~ 0
+Text GLabel 3900 4800 0    50   Input ~ 0
 SCL
-Text GLabel 3950 3550 0    50   Input ~ 0
+Text GLabel 3900 4950 0    50   Input ~ 0
 SDA
 $Comp
@@
 L power:GND #PWR?
 U 1 1 5C816DC7
-P 3800 3100
-F 0 "#PWR?" H 3800 2850 50  0001 C CNN
-F 1 "GND" H 3805 2927 50  0000 C CNN
-F 2 "" H 3800 3100 50  0001 C CNN
-F 3 "" H 3800 3100 50  0001 C CNN
-	1    3800 3100
-	1    0    0    -1
-$EndComp
-Wire Wire Line
-	3800 3100 3950 3100
+P 3750 4500
+F 0 "#PWR?" H 3750 4250 50  0001 C CNN
+F 1 "GND" H 3755 4327 50  0000 C CNN
+F 2 "" H 3750 4500 50  0001 C CNN
+F 3 "" H 3750 4500 50  0001 C CNN
+	1    3750 4500
+	1    0    0    -1
+$EndComp
+Wire Wire Line
+	3750 4500 3900 4500
 $Comp
 L power:GND #PWR?
@@
 Text GLabel 9400 3150 1    50   Input ~ 0
 +5V
-Text GLabel 5050 1750 2    50   Input ~ 0
+Text GLabel 4700 2100 2    50   Input ~ 0
 R_joystick_analog_x
-Text GLabel 5050 1900 2    50   Input ~ 0
+Text GLabel 4700 2250 2    50   Input ~ 0
 R_joystick_analog_y
-Text GLabel 5050 2350 2    50   Input ~ 0
+Text GLabel 3900 3450 0    50   Input ~ 0
 R_joystick_button
-Text GLabel 5050 2050 2    50   Input ~ 0
+Text GLabel 4700 2400 2    50   Input ~ 0
 L_joystick_analog_x
-Text GLabel 5050 2200 2    50   Input ~ 0
+Text GLabel 4700 2550 2    50   Input ~ 0
 L_joystick_analog_y
-Text GLabel 5050 2500 2    50   Input ~ 0
+Text GLabel 3900 3600 0    50   Input ~ 0
 L_joystick_button
-Text GLabel 5050 2800 2    50   Output ~ 0
+Text GLabel 4150 2550 2    50   Input ~ 0
 L_trigger
-Text GLabel 5050 2650 2    50   Output ~ 0
+Text GLabel 4150 2400 2    50   Input ~ 0
 R_trigger
 $Comp
@@
 Text GLabel 2750 3150 2    50   Output ~ 0
 Buzzer
+Text GLabel 3900 3750 0    50   Input ~ 0
+Button_LEFT
+Text GLabel 3900 3900 0    50   Input ~ 0
+Button_UP
+Text GLabel 3900 4050 0    50   Input ~ 0
+Button_RIGHT
+Text GLabel 3900 4200 0    50   Input ~ 0
+Button_DOWN
+Text GLabel 5000 3150 2    50   Input ~ 0
+Button_A
+Text GLabel 5000 3300 2    50   Input ~ 0
+Button_B
+Text GLabel 5000 3450 2    50   Input ~ 0
+Button_Y
+Text GLabel 5000 3600 2    50   Input ~ 0
+Button_X
+Text GLabel 5000 4050 2    50   Input ~ 0
+Button_START
+Text GLabel 5000 4200 2    50   Input ~ 0
+Button_SELECT
+Text GLabel 5000 3750 2    50   Input ~ 0
+R_Bumper
+Text GLabel 5000 3900 2    50   Input ~ 0
+L_Bumper
 $EndSCHEMATC

Commit message: schema
Parts:
- removed J1: Conn_01x10, symbol Connector_Generic:Conn_01x10
- added U?: R-78E5.0-0.5, Converter_DCDC:Converter_DCDC_RECOM_R-78E-0.5_THT, symbol Regulator_Switching:R-78E5.0-0.5
- added U?: ESP32, symbol ESP32:ESP32
- added U?: OLED_Display, symbol Adafruit_OLED_RGB_Screen:OLED_Display
Connections:
- net labels added: Inputs
- wire segments 52 -> 68
Other:
- moved on the sheet: U1

Commit message: update schema
Parts:
- added R4: 200K, symbol Device:R
- added U6: PCA9306, symbol Interface:PCA9306
- added U?: R-783.3-0.5, Converter_DCDC:Converter_DCDC_RECOM_R-78E-0.5_THT, symbol Regulator_Switching:R-783.3-0.5
- D1: renamed from D?; value LED -> LED_B
- D2: renamed from D?; value LED -> LED_R
- SW14: value Power On/Off -> On/Off
- gave numbers to parts that had none: 8
- renumbered U1 to U2, U2 to U3, U3 to U5
Connections:
- net labels added: +3.3V, 3.3V, DC, OLEDCS, Outputs, RX_Atmega, RX_ESP32, SDCS, SerialComm, TX_Atmega, TX_ESP32
- net labels removed: D/C, LCD, SD
- wire segments 68 -> 86
Other:
- moved on the sheet: U2

Commit message: update schéma
Parts:
- RV1: renamed from RV?; value R_POT -> L_trigger
- RV2: renamed from RV?; value R_POT -> R_trigger
- gave numbers to parts that had none: 1
Connections:
- net labels added: Command
- wire segments 86 -> 87
Changed lines of the file:
@@
 encoding utf-8
 Sheet 1 1
-Title "Manette 2019"
+Title "Manette Universelle"
 Date "2019-03-04"
 Rev ""
@@
 $EndComp
 $Comp
-L Device:R_POT RV?
+L Device:R_POT RV1
 U 1 1 5C7D4ACF
 P 8800 6000
-F 0 "RV?" H 8730 6046 50  0000 R CNN
-F 1 "R_POT" H 8730 5955 50  0000 R CNN
+F 0 "RV1" H 8730 6046 50  0000 R CNN
+F 1 "L_trigger" H 8730 5955 50  0000 R CNN
 F 2 "" H 8800 6000 50  0001 C CNN
 F 3 "~" H 8800 6000 50  0001 C CNN
@@
 $EndComp
 $Comp
-L Device:R_POT RV?
+L Device:R_POT RV2
 U 1 1 5C7D4B89
 P 9900 6000
-F 0 "RV?" H 9830 6046 50  0000 R CNN
-F 1 "R_POT" H 9830 5955 50  0000 R CNN
+F 0 "RV2" H 9830 6046 50  0000 R CNN
+F 1 "R_trigger" H 9830 5955 50  0000 R CNN
 F 2 "" H 9900 6000 50  0001 C CNN
 F 3 "~" H 9900 6000 50  0001 C CNN
@@
 $EndComp
 $Comp
-L Device:Speaker LS?
+L Device:Speaker LS1
 U 1 1 5C7D5866
 P 5550 7250
-F 0 "LS?" H 5500 6950 50  0000 L CNN
+F 0 "LS1" H 5500 6950 50  0000 L CNN
 F 1 "Speaker" H 5400 6850 50  0000 L CNN
 F 2 "" H 5550 7050 50  0001 C CNN
@@
 	1    0    0    -1
 $EndComp
-Text GLabel 2750 1900 0    50   Input ~ 0
+Text GLabel 4850 1900 0    50   Input ~ 0
 MISO
-Text GLabel 2750 1800 0    50   Output ~ 0
+Text GLabel 4850 1800 0    50   Output ~ 0
 SCK
-Text GLabel 2750 2000 0    50   Output ~ 0
+Text GLabel 4850 2000 0    50   Output ~ 0
 MOSI
-Text GLabel 2750 1500 0    50   Output ~ 0
+Text GLabel 4850 1500 0    50   Output ~ 0
 RESET
 Text GLabel 3950 5350 2    50   Output ~ 0
@@
 L ESP32:ESP32 U1
 U 1 1 5CA33ACA
-P 3850 1050
-F 0 "U1" H 3850 1525 50  0000 C CNN
-F 1 "ESP32" H 3850 1434 50  0000 C CNN
-F 2 "" H 3250 1000 50  0001 C CNN
-F 3 "" H 3250 1000 50  0001 C CNN
-	1    3850 1050
+P 5950 1050
+F 0 "U1" H 5950 1525 50  0000 C CNN
+F 1 "ESP32" H 5950 1434 50  0000 C CNN
+F 2 "" H 5350 1000 50  0001 C CNN
+F 3 "" H 5350 1000 50  0001 C CNN
+	1    5950 1050
 	1    0    0    -1
 $EndComp
@@
 Text GLabel 1500 6650 0    50   Input ~ 0
 DC
-Text GLabel 2750 1600 0    50   Output ~ 0
+Text GLabel 4850 1600 0    50   Output ~ 0
 DC
 Text GLabel 1500 6850 0    50   Input ~ 0
 OLEDCS
-Text GLabel 2750 1700 0    50   Output ~ 0
+Text GLabel 4850 1700 0    50   Output ~ 0
 OLEDCS
 Text GLabel 3350 2850 1    50   Input ~ 0
@@
 L power:GND #PWR?
 U 1 1 5CA7EA37
-P 2400 2200
-F 0 "#PWR?" H 2400 1950 50  0001 C CNN
-F 1 "GND" H 2405 2027 50  0000 C CNN
-F 2 "" H 2400 2200 50  0001 C CNN
-F 3 "" H 2400 2200 50  0001 C CNN
-	1    2400 2200
-	1    0    0    -1
-$EndComp
-Wire Wire Line
-	2400 2200 2400 2100
-Wire Wire Line
-	2400 2100 2750 2100
-Text GLabel 2750 1400 0    50   Input ~ 0
+P 4500 2200
+F 0 "#PWR?" H 4500 1950 50  0001 C CNN
+F 1 "GND" H 4505 2027 50  0000 C CNN
+F 2 "" H 4500 2200 50  0001 C CNN
+F 3 "" H 4500 2200 50  0001 C CNN
+	1    4500 2200
+	1    0    0    -1
+$EndComp
+Wire Wire Line
+	4500 2200 4500 2100
+Wire Wire Line
+	4500 2100 4850 2100
+Text GLabel 4850 1400 0    50   Input ~ 0
 SDCS
 Text GLabel 1500 6950 0    50   Input ~ 0
@@
 Text Label 650  6300 0    197  ~ 0
 Outputs
-Text GLabel 4950 1100 2    50   Input ~ 0
+Text GLabel 7050 1100 2    50   Input ~ 0
 RX_ESP32
-Text GLabel 4950 1000 2    50   Input ~ 0
+Text GLabel 7050 1000 2    50   Input ~ 0
 TX_ESP32
 $Comp
@@
 	1    0    0    -1
 $EndComp
-Text GLabel 2750 2200 0    50   Input ~ 0
+Text GLabel 4850 2200 0    50   Input ~ 0
 +3.3V
 Text GLabel 1500 3100 1    50   Input ~ 0
@@
 Wire Notes Line
 	500  2550 2300 2550
-Text Label 750  700  0    197  ~ 0
+Text Label 750  750  0    197  ~ 0
 Power
 Wire Notes Line
@@
 Text Label 500  2800 0    197  ~ 0
 SerialComm
+Text Label 2550 750  0    197  ~ 0
+Command
+Text GLabel 5600 5050 2    50   Output ~ 0
++5V
+Wire Wire Line
+	7850 4000 7750 4000
 $EndSCHEMATC
