File: 07_Schémas/manette_2019/manette_2019.sch (KiCad schematic (older format))
At the start: 35 parts, among them SW1 Button_A, SW10 Button_DOWN, SW11 R_bumper, SW12 L_bumper, SW13 Calib, SW14 On/Off, SW2 Button_B, SW3 Button_X, SW4 Button_Y, SW5 Button_START, SW6 Button_SELECT, SW7 Button_RIGHT, SW8 Button_UP, SW9 Button_LEFT, U1 ESP32, U2 ATmega328-PU, U3 MCP23017, U4 OLED_Display, U5 ULN2803A, U6 PCA9306, U6 R-78E5.0-0.5, Y1 Resonator

Commit message: update schema
Parts:
- added J1: Power, TerminalBlock:TerminalBlock_bornier-2_P5.08mm, symbol Connector:Screw_Terminal_01x02
- D1, D2: footprint (none) -> LED_THT:LED_D3.0mm
- D3: footprint (none) -> Diode_THT:D_A-405_P10.16mm_Horizontal
- JS1, JS2: footprint (none) -> Polymanette_2018:Joystick_RSF_2-axis
- LS1: footprint (none) -> Buzzer_Beeper:Buzzer_T135
- R1, R2, R3: footprint (none) -> Resistor_THT:R_Axial_DIN0309_L9.0mm_D3.2mm_P15.24mm_Horizontal
- U1: footprint (none) -> ESP32:ESP32
- U3: footprint (none) -> Package_DIP:DIP-28_W7.62mm
- U5: footprint (none) -> Package_DIP:DIP-18_W7.62mm
- gave numbers to parts that had none: 1
- renumbered U6 to U7, U6 to U8
Connections:
- net labels added: +10V
- wire segments 87 -> 91
Other:
- moved on the sheet: U2, U6

Commit message: update
Parts:
- removed U4: OLED_Display, symbol Adafruit_OLED_RGB_Screen:OLED_Display
- added U4: OLED_Display, symbol OLED:OLED_Display
- SW1, SW10, SW11, SW12, SW2, SW3, SW4, SW5, SW6, SW7, SW8, SW9: footprint (none) -> Button_Switch_THT:Bouton_MEC
Connections:
- net labels added: Calib
Changed lines of the file:
@@
 F 0 "SW3" H 10700 2335 50  0000 C CNN
 F 1 "Button_X" H 10700 2244 50  0000 C CNN
-F 2 "" H 10700 2250 50  0001 C CNN
+F 2 "Button_Switch_THT:Bouton_MEC" H 10700 2250 50  0001 C CNN
 F 3 "" H 10700 2250 50  0001 C CNN
 	1    10700 2050
@@
 F 0 "SW4" H 10700 2685 50  0000 C CNN
 F 1 "Button_Y" H 10700 2594 50  0000 C CNN
-F 2 "" H 10700 2600 50  0001 C CNN
+F 2 "Button_Switch_THT:Bouton_MEC" H 10700 2600 50  0001 C CNN
 F 3 "" H 10700 2600 50  0001 C CNN
 	1    10700 2400
@@
 F 0 "SW5" H 10700 3035 50  0000 C CNN
 F 1 "Button_START" H 10700 2944 50  0000 C CNN
-F 2 "" H 10700 2950 50  0001 C CNN
+F 2 "Button_Switch_THT:Bouton_MEC" H 10700 2950 50  0001 C CNN
 F 3 "" H 10700 2950 50  0001 C CNN
 	1    10700 2750
@@
 F 0 "SW6" H 10700 3385 50  0000 C CNN
 F 1 "Button_SELECT" H 10700 3294 50  0000 C CNN
-F 2 "" H 10700 3300 50  0001 C CNN
+F 2 "Button_Switch_THT:Bouton_MEC" H 10700 3300 50  0001 C CNN
 F 3 "" H 10700 3300 50  0001 C CNN
 	1    10700 3100
@@
 F 0 "SW11" H 10700 5235 50  0000 C CNN
 F 1 "R_bumper" H 10700 5144 50  0000 C CNN
-F 2 "" H 10700 5150 50  0001 C CNN
+F 2 "Button_Switch_THT:Bouton_MEC" H 10700 5150 50  0001 C CNN
 F 3 "" H 10700 5150 50  0001 C CNN
 	1    10700 4950
@@
 F 0 "SW9" H 10700 4535 50  0000 C CNN
 F 1 "Button_LEFT" H 10700 4444 50  0000 C CNN
-F 2 "" H 10700 4450 50  0001 C CNN
+F 2 "Button_Switch_THT:Bouton_MEC" H 10700 4450 50  0001 C CNN
 F 3 "" H 10700 4450 50  0001 C CNN
 	1    10700 4250
@@
 F 0 "SW10" H 10700 4885 50  0000 C CNN
 F 1 "Button_DOWN" H 10700 4794 50  0000 C CNN
-F 2 "" H 10700 4800 50  0001 C CNN
+F 2 "Button_Switch_THT:Bouton_MEC" H 10700 4800 50  0001 C CNN
 F 3 "" H 10700 4800 50  0001 C CNN
 	1    10700 4600
@@
 F 0 "SW1" H 10700 1635 50  0000 C CNN
 F 1 "Button_A" H 10700 1544 50  0000 C CNN
-F 2 "" H 10700 1550 50  0001 C CNN
+F 2 "Button_Switch_THT:Bouton_MEC" H 10700 1550 50  0001 C CNN
 F 3 "" H 10700 1550 50  0001 C CNN
 	1    10700 1350
@@
 F 0 "SW2" H 10700 1985 50  0000 C CNN
 F 1 "Button_B" H 10700 1894 50  0000 C CNN
-F 2 "" H 10700 1900 50  0001 C CNN
+F 2 "Button_Switch_THT:Bouton_MEC" H 10700 1900 50  0001 C CNN
 F 3 "" H 10700 1900 50  0001 C CNN
 	1    10700 1700
@@
 F 0 "SW7" H 10700 3735 50  0000 C CNN
 F 1 "Button_RIGHT" H 10700 3644 50  0000 C CNN
-F 2 "" H 10700 3650 50  0001 C CNN
+F 2 "Button_Switch_THT:Bouton_MEC" H 10700 3650 50  0001 C CNN
 F 3 "" H 10700 3650 50  0001 C CNN
 	1    10700 3450
@@
 F 0 "SW8" H 10700 4135 50  0000 C CNN
 F 1 "Button_UP" H 10700 4044 50  0000 C CNN
-F 2 "" H 10700 4050 50  0001 C CNN
+F 2 "Button_Switch_THT:Bouton_MEC" H 10700 4050 50  0001 C CNN
 F 3 "" H 10700 4050 50  0001 C CNN
 	1    10700 3850
@@
 F 0 "SW12" H 10700 5585 50  0000 C CNN
 F 1 "L_bumper" H 10700 5494 50  0000 C CNN
-F 2 "" H 10700 5500 50  0001 C CNN
+F 2 "Button_Switch_THT:Bouton_MEC" H 10700 5500 50  0001 C CNN
 F 3 "" H 10700 5500 50  0001 C CNN
 	1    10700 5300
@@
 Text GLabel 10500 4600 0    50   Input ~ 0
 Button_DOWN
-$Comp
-L ESP32:ESP32 U1
-U 1 1 5CA33ACA
-P 5950 1050
-F 0 "U1" H 5950 1525 50  0000 C CNN
-F 1 "ESP32" H 5950 1434 50  0000 C CNN
-F 2 "ESP32:ESP32" H 5350 1000 50  0001 C CNN
-F 3 "" H 5350 1000 50  0001 C CNN
-	1    5950 1050
-	1    0    0    -1
-$EndComp
 Text Label 9850 800  0    197  ~ 0
 Inputs
-$Comp
-L Adafruit_OLED_RGB_Screen:OLED_Display U4
-U 1 1 5CA3C6B3
-P 1800 7000
-F 0 "U4" H 2028 7076 50  0000 L CNN
-F 1 "OLED_Display" H 2028 6985 50  0000 L CNN
-F 2 "" H 1800 7000 50  0001 C CNN
-F 3 "" H 1800 7000 50  0001 C CNN
-	1    1800 7000
-	1    0    0    -1
-$EndComp
 Text GLabel 1500 6650 0    50   Input ~ 0
 DC
@@
 Wire Wire Line
 	1100 1225 1100 1325
+Text GLabel 5825 3175 0    50   Output ~ 0
+Calib
+Text GLabel 10500 5650 0    50   Input ~ 0
+Calib
+$Comp
+L ESP32:ESP32 U1
+U 1 1 5CABDA52
+P 5950 1050
+F 0 "U1" H 5950 1525 50  0000 C CNN
+F 1 "ESP32" H 5950 1434 50  0000 C CNN
+F 2 "ESP32:ESP32" H 5350 1000 50  0001 C CNN
+F 3 "" H 5350 1000 50  0001 C CNN
+	1    5950 1050
+	1    0    0    -1
+$EndComp
+$Comp
+L OLED:OLED_Display U4
+U 1 1 5CAC3235
+P 1800 7000
+F 0 "U4" H 2028 7076 50  0000 L CNN
+F 1 "OLED_Display" H 2028 6985 50  0000 L CNN
+F 2 "" H 1800 7000 50  0001 C CNN
+F 3 "" H 1800 7000 50  0001 C CNN
+	1    1800 7000
+	1    0    0    -1
+$EndComp
 $EndSCHEMATC

Commit message: update
Parts:
- removed R4: 200K, symbol Device:R
- removed RV1: L_trigger, symbol Device:R_POT
- removed RV2: R_trigger, symbol Device:R_POT
- removed SW11: R_bumper, Button_Switch_THT:Bouton_MEC, symbol Switch:SW_Push
- removed SW12: L_bumper, Button_Switch_THT:Bouton_MEC, symbol Switch:SW_Push
- removed SW14: On/Off, symbol Switch:SW_DPST_x2
- removed U8: PCA9306, symbol Interface:PCA9306
- added J2: Screw_Terminal_01x06, TerminalBlock:TerminalBlock_bornier-6_P5.08mm, symbol Connector:Screw_Terminal_01x06
- added U8: PCA9306, PCA9306:PCA9306, symbol PCA9306:PCA9306
- U4: footprint (none) -> OLED:OLED RGB
- Y1: footprint (none) -> Crystal:Resonator-3Pin_W6.0mm_H3.0mm
Connections:
- wire segments 91 -> 85

Commit message: update
Parts:
- removed J2: Screw_Terminal_01x06, TerminalBlock:TerminalBlock_bornier-6_P5.08mm, symbol Connector:Screw_Terminal_01x06
- added C1, C2, C3, C4, C5, C6: C, Capacitor_THT:C_Disc_D5.0mm_W2.5mm_P5.00mm, symbol Device:C
- added J2, J3: Screw_Terminal_01x04, TerminalBlock:TerminalBlock_bornier-4_P5.08mm, symbol Connector:Screw_Terminal_01x04
- added R4: R, Resistor_THT:R_Axial_DIN0309_L9.0mm_D3.2mm_P15.24mm_Horizontal, symbol Device:R
- JS1: value Joystick_RSF_2-Axis -> Joystick_Left
- JS2: value Joystick_RSF_2-Axis -> Joystick_Right
- SW13: footprint (none) -> Button_Switch_THT:Bouton_MEC
Connections:
- net labels added: +9V
- net labels removed: +10V, 3.3V
- wire segments 85 -> 107
- no-connect marks 0 -> 48

Commit message: a
Parts:
- removed U4: OLED_Display, OLED:OLED RGB, symbol OLED:OLED_Display
- added C7, C8, C9: C, symbol Device:C
- added J4: OLED_Display, TerminalBlock_4Ucon:TerminalBlock_4Ucon_1x09_P3.50mm_Horizontal, symbol Connector:Screw_Terminal_01x09
- C1, C2, C3, C4, C5, C6: footprint Capacitor_THT:C_Disc_D5.0mm_W2.5mm_P5.00mm -> (none)
Connections:
- net labels added: VCC, Vcc_Atmega328P, Vcc_Bus, Vcc_ESP32, Vcc_Left_Js, Vcc_OLED_Display, Vcc_Rec_3.3, Vcc_Rec_5, Vcc_Right_Js
- net labels removed: +9V
- wire segments 107 -> 103
- no-connect marks 48 -> 46
Other:
- moved on the sheet: U2, U6

Commit message: update schema
Parts:
- added D4: D, Diode_THT:D_A-405_P10.16mm_Horizontal, symbol Device:D
- added J5: Rumble, symbol Connector:Screw_Terminal_01x02
- added R?: R, Resistor_THT:R_Axial_DIN0309_L9.0mm_D3.2mm_P15.24mm_Horizontal, symbol Device:R
- C1, C2, C3, C4, C5, C6, C7, C8: footprint (none) -> Capacitor_THT:C_Rect_L7.0mm_W3.5mm_P5.00mm
- C9: footprint (none) -> Capacitor_THT:C_Radial_D10.0mm_H20.0mm_P5.00mm
Connections:
- net labels added: Rumble
- wire segments 103 -> 109
- no-connect marks 46 -> 44

Commit message: Plans et data movement
Parts:
- removed C4, C5: C, Capacitor_THT:C_Rect_L7.0mm_W3.5mm_P5.00mm, symbol Device:C
- removed D1: LED_B, LED_THT:LED_D3.0mm, symbol Device:LED
- removed D2: LED_R, LED_THT:LED_D3.0mm, symbol Device:LED
- removed J2, J3: Screw_Terminal_01x04, TerminalBlock:TerminalBlock_bornier-4_P5.08mm, symbol Connector:Screw_Terminal_01x04
- removed J4: OLED_Display, TerminalBlock_4Ucon:TerminalBlock_4Ucon_1x09_P3.50mm_Horizontal, symbol Connector:Screw_Terminal_01x09
- removed R1, R2: R, Resistor_THT:R_Axial_DIN0309_L9.0mm_D3.2mm_P15.24mm_Horizontal, symbol Device:R
- removed SW1: Button_A, Button_Switch_THT:Bouton_MEC, symbol Switch:SW_Push
- removed SW10: Button_DOWN, Button_Switch_THT:Bouton_MEC, symbol Switch:SW_Push
- removed SW13: Calib, Button_Switch_THT:Bouton_MEC, symbol Manette_arcade:SW_Push
- removed SW2: Button_B, Button_Switch_THT:Bouton_MEC, symbol Switch:SW_Push
- removed SW3: Button_X, Button_Switch_THT:Bouton_MEC, symbol Switch:SW_Push
- removed SW4: Button_Y, Button_Switch_THT:Bouton_MEC, symbol Switch:SW_Push
- removed SW5: Button_START, Button_Switch_THT:Bouton_MEC, symbol Switch:SW_Push
- removed SW6: Button_SELECT, Button_Switch_THT:Bouton_MEC, symbol Switch:SW_Push
- removed SW7: Button_RIGHT, Button_Switch_THT:Bouton_MEC, symbol Switch:SW_Push
- removed SW8: Button_UP, Button_Switch_THT:Bouton_MEC, symbol Switch:SW_Push
- removed SW9: Button_LEFT, Button_Switch_THT:Bouton_MEC, symbol Switch:SW_Push
- added J10: Alim_LED, TerminalBlock:TerminalBlock_bornier-2_P5.08mm, symbol Connector:Screw_Terminal_01x02
- added J2: L_Bumper, Connector_PinSocket_2.54mm:PinSocket_1x02_P2.54mm_Vertical, symbol Connector_Generic:Conn_01x02
- added J3: R_Bumper, Connector_PinSocket_2.54mm:PinSocket_1x02_P2.54mm_Vertical, symbol Connector_Generic:Conn_01x02
- added J4: OLED_Display, Connector_PinSocket_2.54mm:PinSocket_1x09_P2.54mm_Vertical, symbol Connector_Generic:Conn_01x09
- added J6: Calib, Connector_PinSocket_2.54mm:PinSocket_1x02_P2.54mm_Vertical, symbol Connector_Generic:Conn_01x02
- added J7: Conn_R_Button, manette_2019:Conn_8, symbol Connector_Generic:Conn_01x08
- added J8: Conn_L_Button, manette_2019:Conn_8, symbol Connector_Generic:Conn_01x08
- added J9: Conn_Middle_PCB, manette_2019:Conn_8, symbol Connector_Generic:Conn_01x08
- added RV1, RV2: R_POT, Potentiometer_THT:Potentiometer_Bourns_PTA2043_Single_Slide, symbol Device:R_POT
- J1: value Power -> Vcc
- J5: footprint (none) -> TerminalBlock:TerminalBlock_bornier-2_P5.08mm
- U1: footprint ESP32:ESP32 -> manette_2019:ESP32
- U8: footprint PCA9306:PCA9306 -> manette_2019:PCA9306
- gave numbers to parts that had none: 1
- renumbered C9 to C1, C1 to C2, C8 to C3, C7 to C4, C2 to C5, C3 to C6, C6 to C7
Connections:
- net labels added: Conn_LED_On, VCC_LED
- net labels removed: L_joystick_button, Left_trigger, R_joystick_button, Right_trigger, Vcc_Atmega328P, Vcc_Bus, Vcc_ESP32, Vcc_Left_Js, Vcc_OLED_Display, Vcc_Rec_3.3, Vcc_Rec_5, Vcc_Right_Js
- wire segments 109 -> 97
- no-connect marks 44 -> 52
Other:
- moved on the sheet: U2

Commit message: update
Parts:
- removed C3, C4: C, Capacitor_THT:C_Rect_L7.0mm_W3.5mm_P5.00mm, symbol Device:C
- removed U6: R-783.3-0.5, Converter_DCDC:Converter_DCDC_RECOM_R-78E-0.5_THT, symbol Regulator_Switching:R-783.3-0.5
- removed U7: R-78E5.0-0.5, Converter_DCDC:Converter_DCDC_RECOM_R-78E-0.5_THT, symbol Regulator_Switching:R-78E5.0-0.5
Connections:
- net labels removed: VCC
- wire segments 97 -> 92
- no-connect marks 52 -> 51
Changed lines of the file:
@@
 Wire Wire Line
 	7150 3725 7050 3725
-Text GLabel 2375 2325 2    50   Output ~ 0
-+5V
 $Comp
 L power:GND #PWR0111
@@
 Text GLabel 6100 1625 0    50   Input ~ 0
 Button_LEFT
-Text GLabel 6100 1475 0    50   Input ~ 0
+Text GLabel 6100 1175 0    50   Input ~ 0
 Button_UP
 Text GLabel 6100 1325 0    50   Input ~ 0
 Button_RIGHT
-Text GLabel 6100 1175 0    50   Input ~ 0
+Text GLabel 6100 1475 0    50   Input ~ 0
 Button_DOWN
-Text GLabel 7200 1475 2    50   Input ~ 0
+Text GLabel 7200 1175 2    50   Input ~ 0
 Button_A
 Text GLabel 7200 1325 2    50   Input ~ 0
 Button_B
-Text GLabel 7200 1175 2    50   Input ~ 0
+Text GLabel 7200 1475 2    50   Input ~ 0
 Button_Y
 Text GLabel 7200 1025 2    50   Input ~ 0
@@
 Wire Wire Line
 	6500 3775 6150 3775
-$Comp
-L Regulator_Switching:R-78E5.0-0.5 U7
-U 1 1 5C9AC915
-P 2075 2325
-F 0 "U7" H 2075 2567 50  0000 C CNN
-F 1 "R-78E5.0-0.5" H 2075 2476 50  0000 C CNN
-F 2 "Converter_DCDC:Converter_DCDC_RECOM_R-78E-0.5_THT" H 2125 2075 50  0001 L CIN
-F 3 "https://www.recom-power.com/pdf/Innoline/R-78Exx-0.5.pdf" H 2075 2325 50  0001 C CNN
-	1    2075 2325
-	1    0    0    -1
-$EndComp
-$Comp
-L power:GND #PWR0112
-U 1 1 5C9B9F3C
-P 2075 2625
-F 0 "#PWR0112" H 2075 2375 50  0001 C CNN
-F 1 "GND" H 2080 2452 50  0000 C CNN
-F 2 "" H 2075 2625 50  0001 C CNN
-F 3 "" H 2075 2625 50  0001 C CNN
-	1    2075 2625
-	1    0    0    -1
-$EndComp
 Text Label 1725 3150 0    197  ~ 0
 Inputs
@@
 Text GLabel 9700 3175 0    50   Input ~ 0
 RX_Atmega
-$Comp
-L Regulator_Switching:R-783.3-0.5 U6
-U 1 1 5CB0E72E
-P 2075 1475
-F 0 "U6" H 2075 1717 50  0000 C CNN
-F 1 "R-783.3-0.5" H 2075 1626 50  0000 C CNN
-F 2 "Converter_DCDC:Converter_DCDC_RECOM_R-78E-0.5_THT" H 2125 1225 50  0001 L CIN
-F 3 "https://www.recom-power.com/pdf/Innoline/R-78xx-0.5.pdf" H 2075 1475 50  0001 C CNN
-	1    2075 1475
-	1    0    0    -1
-$EndComp
-$Comp
-L power:GND #PWR0117
-U 1 1 5CB1A915
-P 2075 1775
-F 0 "#PWR0117" H 2075 1525 50  0001 C CNN
-F 1 "GND" H 2080 1602 50  0000 C CNN
-F 2 "" H 2075 1775 50  0001 C CNN
-F 3 "" H 2075 1775 50  0001 C CNN
-	1    2075 1775
-	1    0    0    -1
-$EndComp
-Text GLabel 2375 1475 2    50   Output ~ 0
-+3.3V
 Text Label 1050 725  0    197  ~ 0
 Power
@@
 Connected
 Text GLabel 1325 1100 2    50   Output ~ 0
-VCC
-$Comp
-L power:PWR_FLAG #FLG0101
-U 1 1 5CA7532E
-P 6350 6400
-F 0 "#FLG0101" H 6350 6475 50  0001 C CNN
-F 1 "PWR_FLAG" H 6350 6574 50  0000 C CNN
-F 2 "" H 6350 6400 50  0001 C CNN
-F 3 "~" H 6350 6400 50  0001 C CNN
-	1    6350 6400
-	1    0    0    -1
-$EndComp
++5V
 $Comp
 L power:PWR_FLAG #FLG0102
@@
 Text GLabel 6525 6400 3    50   Input ~ 0
 +5V
-Text GLabel 6350 6400 3    50   Input ~ 0
-VCC
 $Comp
 L power:GND #PWR0102
@@
 $EndComp
 Text GLabel 11150 4975 1    50   Input ~ 0
-VCC
++5V
 NoConn ~ 5825 3175
 NoConn ~ 6150 3275
@@
 NoConn ~ 8550 900
 NoConn ~ 8550 800
-NoConn ~ 10750 2200
 NoConn ~ 10750 2100
 NoConn ~ 10750 2000
@@
 Wire Notes Line
 	4725 6100 4725 475
-Text GLabel 3375 6400 1    50   Input ~ 0
-VCC
+Text GLabel 3975 6400 1    50   Input ~ 0
++5V
 $Comp
 L Device:C C5
 U 1 1 5CC5B24F
-P 4850 6725
-F 0 "C5" H 4965 6771 50  0000 L CNN
-F 1 "C" H 4965 6680 50  0000 L CNN
-F 2 "Capacitor_THT:C_Rect_L7.0mm_W3.5mm_P5.00mm" H 4888 6575 50  0001 C CNN
-F 3 "Vin_Bus" H 5025 6600 50  0000 C CNN
-	1    4850 6725
-	1    0    0    -1
-$EndComp
-Text GLabel 4850 6400 1    50   Input ~ 0
-+5V
+P 3775 6725
+F 0 "C5" H 3890 6771 50  0000 L CNN
+F 1 "C" H 3890 6680 50  0000 L CNN
+F 2 "Capacitor_THT:C_Rect_L7.0mm_W3.5mm_P5.00mm" H 3813 6575 50  0001 C CNN
+F 3 "Vin_Bus" H 3950 6600 50  0000 C CNN
+	1    3775 6725
+	1    0    0    -1
+$EndComp
 Wire Wire Line
 	7950 2100 8550 2100
@@
 L Device:C C6
 U 1 1 5CCA67BF
-P 5250 6725
-F 0 "C6" H 5365 6771 50  0000 L CNN
-F 1 "C" H 5365 6680 50  0000 L CNN
-F 2 "Capacitor_THT:C_Rect_L7.0mm_W3.5mm_P5.00mm" H 5288 6575 50  0001 C CNN
-F 3 "Vin_Atmega" H 5475 6600 50  0000 C CNN
-	1    5250 6725
+P 4175 6725
+F 0 "C6" H 4290 6771 50  0000 L CNN
+F 1 "C" H 4290 6680 50  0000 L CNN
+F 2 "Capacitor_THT:C_Rect_L7.0mm_W3.5mm_P5.00mm" H 4213 6575 50  0001 C CNN
+F 3 "Vin_Atmega" H 4400 6600 50  0000 C CNN
+	1    4175 6725
 	1    0    0    -1
 $EndComp
@@
 L Device:C C7
 U 1 1 5CCE01FA
-P 5775 6725
-F 0 "C7" H 5890 6771 50  0000 L CNN
-F 1 "C" H 5890 6680 50  0000 L CNN
-F 2 "Capacitor_THT:C_Rect_L7.0mm_W3.5mm_P5.00mm" H 5813 6575 50  0001 C CNN
-F 3 "Vin_OLED_Display" H 6125 6600 50  0000 C CNN
-	1    5775 6725
-	1    0    0    -1
-$EndComp
-Text GLabel 5775 6400 1    50   Input ~ 0
-+3.3V
-$Comp
-L Device:C C4
-U 1 1 5CD26113
-P 4350 6725
-F 0 "C4" H 4465 6771 50  0000 L CNN
-F 1 "C" H 4465 6680 50  0000 L CNN
-F 2 "Capacitor_THT:C_Rect_L7.0mm_W3.5mm_P5.00mm" H 4388 6575 50  0001 C CNN
-F 3 "Vin_Rec_U7" H 4575 6600 50  0000 C CNN
-	1    4350 6725
-	1    0    0    -1
-$EndComp
-$Comp
-L Device:C C3
-U 1 1 5CD5092B
-P 3825 6725
-F 0 "C3" H 3940 6771 50  0000 L CNN
-F 1 "C" H 3940 6680 50  0000 L CNN
-F 2 "Capacitor_THT:C_Rect_L7.0mm_W3.5mm_P5.00mm" H 3863 6575 50  0001 C CNN
-F 3 "Vin_Rec_U6" H 4100 6600 50  0000 C CNN
-	1    3825 6725
+P 4725 6725
+F 0 "C7" H 4840 6771 50  0000 L CNN
+F 1 "C" H 4840 6680 50  0000 L CNN
+F 2 "Capacitor_THT:C_Rect_L7.0mm_W3.5mm_P5.00mm" H 4763 6575 50  0001 C CNN
+F 3 "Vin_OLED_Display" H 5075 6600 50  0000 C CNN
+	1    4725 6725
 	1    0    0    -1
 $EndComp
@@
 Text GLabel 3850 4775 0    50   Output ~ 0
 Button_LEFT
-Text GLabel 3850 4575 0    50   Output ~ 0
+Text GLabel 3850 4175 0    50   Output ~ 0
 Button_UP
 Text GLabel 3850 4375 0    50   Output ~ 0
 Button_RIGHT
-Text GLabel 3850 4175 0    50   Output ~ 0
+Text GLabel 3850 4575 0    50   Output ~ 0
 Button_DOWN
 Wire Wire Line
@@
 Text GLabel 3850 3225 0    50   Output ~ 0
 Button_B
+Text GLabel 3850 3425 0    50   Output ~ 0
+Button_A
 Text GLabel 3850 3025 0    50   Output ~ 0
-Button_A
-Text GLabel 3850 3425 0    50   Output ~ 0
 Button_Y
 Text GLabel 3850 3625 0    50   Output ~ 0
 Button_X
 Text GLabel 8550 2200 0    50   Input ~ 0
-VCC
-Text GLabel 1775 2325 0    50   Input ~ 0
-VCC
-Text GLabel 1775 1475 0    50   Input ~ 0
-VCC
++5V
 Text GLabel 850  5875 1    50   Input ~ 0
 +5V
@@
 Text GLabel 6100 2075 0    50   Input ~ 0
 +5V
-Text GLabel 9050 4425 0    50   Input ~ 0
-+3.3V
 Wire Wire Line
 	3375 6875 3375 7000
 Wire Wire Line
-	3375 7000 3825 7000
-Wire Wire Line
-	3825 7000 3825 6875
-Connection ~ 3825 7000
-Wire Wire Line
-	4850 7000 4850 6875
-Wire Wire Line
-	5250 7000 5250 6875
-Wire Wire Line
-	5775 7000 5775 6875
-Wire Wire Line
-	3375 6400 3375 6475
-Wire Wire Line
-	3375 6475 3825 6475
-Wire Wire Line
-	3825 6475 3825 6575
-Connection ~ 3375 6475
+	3775 7000 3775 6875
+Wire Wire Line
+	4175 7000 4175 6875
+Wire Wire Line
+	3975 6400 3975 6475
 Wire Wire Line
 	3375 6475 3375 6575
-Connection ~ 3825 6475
-Wire Wire Line
-	4850 6400 4850 6475
-Wire Wire Line
-	5250 6475 4850 6475
-Wire Wire Line
-	5250 6475 5250 6575
-Connection ~ 4850 6475
-Wire Wire Line
-	4850 6475 4850 6575
 $Comp
 L power:GND #PWR0107
 U 1 1 5CCF972D
-P 4350 7000
-F 0 "#PWR0107" H 4350 6750 50  0001 C CNN
-F 1 "GND" H 4355 6827 50  0000 C CNN
-F 2 "" H 4350 7000 50  0001 C CNN
-F 3 "" H 4350 7000 50  0001 C CNN
-	1    4350 7000
-	1    0    0    -1
-$EndComp
-Connection ~ 4350 7000
-Wire Wire Line
-	3825 7000 4350 7000
-Wire Wire Line
-	4350 7000 4350 6875
-Wire Wire Line
-	4350 6575 4350 6475
-Wire Wire Line
-	3825 6475 4350 6475
-Wire Wire Line
-	4350 7000 4850 7000
-Connection ~ 4850 7000
-Wire Wire Line
-	4850 7000 5250 7000
-Wire Wire Line
-	5250 7000 5775 7000
-Connection ~ 5250 7000
-Wire Wire Line
-	5775 6400 5775 6575
+P 3675 7000
+F 0 "#PWR0107" H 3675 6750 50  0001 C CNN
+F 1 "GND" H 3680 6827 50  0000 C CNN
+F 2 "" H 3675 7000 50  0001 C CNN
+F 3 "" H 3675 7000 50  0001 C CNN
+	1    3675 7000
+	1    0    0    -1
+$EndComp
 $Comp
 L Device:C C1
@@
 $EndComp
 Text GLabel 3500 2100 0    50   Input ~ 0
-VCC
++5V
 Text GLabel 9950 6025 2    50   Output ~ 0
 Conn_LED_On
@@
 Wire Wire Line
 	3250 4075 3850 4075
+Wire Wire Line
+	3775 6475 3775 6575
+Wire Wire Line
+	4175 6475 4175 6575
+Wire Wire Line
+	4725 7000 4725 6875
+Wire Wire Line
+	4725 6575 4725 6475
+Text GLabel 9050 4425 0    50   Input ~ 0
++5V
+Wire Wire Line
+	3375 7000 3675 7000
+Wire Wire Line
+	3375 6475 3775 6475
+Connection ~ 3675 7000
+Wire Wire Line
+	3675 7000 3775 7000
+Connection ~ 3775 6475
+Wire Wire Line
+	3775 6475 3975 6475
+Connection ~ 3775 7000
+Wire Wire Line
+	3775 7000 4175 7000
+Connection ~ 4175 6475
+Connection ~ 4175 7000
+Wire Wire Line
+	4175 7000 4725 7000
+Connection ~ 3975 6475
+Wire Wire Line
+	3975 6475 4175 6475
+Wire Wire Line
+	4175 6475 4725 6475
+Text GLabel 10750 2200 2    50   Output ~ 0
++3.3V
 $EndSCHEMATC
