File: 07_Schémas/manette_2019/manette_2019.kicad_pcb (KiCad board)
At the start: 2 copper layers, 150 x 100 mm, 39 parts, among them J1 Vcc, J10 Alim_LED, J2 L_Bumper, J3 R_Bumper, J4 OLED_Display, J5 Rumble, J6 Calib, J7 Conn_01x06, J8 Conn_01x06, J9 Conn_01x05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

Commit message: update schema
Parts:
- removed the REF** at (183.2, 16.3)
- removed the REF** at (172.3, 86.9)
- removed the REF** at (-32.8, 2.48)
- added REF**: MountingHole_3.2mm_M3, MountingHole:MountingHole_3.2mm_M3, F.Cu at (114.3, 81.3)
- added REF**: MountingHole_3.2mm_M3, MountingHole:MountingHole_3.2mm_M3, F.Cu at (73.7, 20.6)
- J7: value Conn_01x06 -> Conn_R_Button; footprint Connector_PinHeader_2.54mm:PinHeader_1x06_P2.54mm_Vertical -> manette_2019:Conn_8
- J8: value Conn_01x06 -> Conn_L_Button; footprint Connector_PinHeader_2.54mm:PinHeader_1x06_P2.54mm_Vertical -> manette_2019:Conn_8
- J9: value Conn_01x05 -> Conn_Middle_PCB; footprint Connector_PinHeader_2.54mm:PinHeader_1x05_P2.54mm_Vertical -> manette_2019:Conn_8
- moved J8 187.8 mm to (8.64, 61.5), turned to 270 degrees
- moved J7 60.6 mm to (134.9, 55.9), turned to 90 degrees
- moved REF** 25.5 mm to (8.00, 82.0)
- moved J9 25.2 mm to (75.8, 52.0)
- moved J4 18.6 mm to (46.0, 15.7)
- moved J2 1.83 mm to (57.1, 5.00)
- moved J3 1.03 mm to (94.0, 4.00)
Connections:
- J7 pad 2: GND -> Button_X
- J7 pad 3: Button_X -> GND
- J7 pad 5: Button_B -> Net-(J7-Pad5)
- J7 pad 6: Button_A -> Button_B
- J8 pad 2: GND -> Button_LEFT
- J8 pad 3: Button_LEFT -> GND
- J8 pad 5: Button_RIGHT -> Net-(J8-Pad5)
- J8 pad 6: Button_DOWN -> Button_RIGHT
- J9 pad 1: GND -> Button_SELECT
- J9 pad 2: Button_SELECT -> Conn_LED_On
- J9 pad 4: VCC -> Net-(J9-Pad4)
- J9 pad 5: Conn_LED_On -> Net-(J9-Pad5)
Routing:
- net VCC_LED: track 0.00 -> 219.4 mm
- net +5V: track 459.0 -> 579.6 mm
- net Button_DOWN: track 0.00 -> 118.4 mm
- net Button_RIGHT: track 0.00 -> 117.0 mm
- net Button_UP: track 0.00 -> 115.3 mm
- net Button_LEFT: track 0.00 -> 113.8 mm
- net Button_B: track 0.00 -> 71.0 mm
- net Button_A: track 0.00 -> 71.0 mm
- net Button_Y: track 0.00 -> 70.4 mm
- net Button_X: track 0.00 -> 69.8 mm
- net Button_SELECT: track 0.00 -> 38.4 mm
- net Button_START: track 0.00 -> 35.8 mm
- net GND: track 725.8 -> 760.3 mm
- net MISO: track 97.3 -> 75.0 mm
- net SDCS: track 69.0 -> 49.7 mm
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- added copper zone on F.Cu, net GND
- added copper zone on B.Cu, net VCC
Other:
- outline, holes or cut-outs redrawn
- net class Default: trace_width 0.25 -> 0.5

Commit message: update
Connections:
- J7 pad 1: VCC_LED -> GND
- J7 pad 2: Button_X -> Button_A
- J7 pad 3: GND -> VCC_LED
- J7 pad 4: Button_Y -> Button_B
- J7 pad 6: Button_B -> Button_Y
- J7 pad 8: Button_A -> Button_X
- J8 pad 1: VCC_LED -> GND
- J8 pad 2: Button_LEFT -> Button_DOWN
- J8 pad 3: GND -> VCC_LED
- J8 pad 4: Button_UP -> Button_RIGHT
- J8 pad 6: Button_RIGHT -> Button_UP
- J8 pad 8: Button_DOWN -> Button_LEFT
- U3 pad 24: Button_X -> Button_A
- U3 pad 25: Button_Y -> Button_B
- U3 pad 26: Button_B -> Button_Y
- U3 pad 27: Button_A -> Button_X
- U3 pad 3: Button_LEFT -> Button_DOWN
- U3 pad 4: Button_UP -> Button_RIGHT
- U3 pad 5: Button_RIGHT -> Button_UP
- U3 pad 6: Button_DOWN -> Button_LEFT
Routing:
- net GND: track 760.3 -> 754.7 mm
- net Button_LEFT: track 113.8 -> 118.4 mm
- net Button_DOWN: track 118.4 -> 113.8 mm
- net Button_UP: track 115.3 -> 117.0 mm
- net Button_RIGHT: track 117.0 -> 115.3 mm
- net VCC_LED: track 219.4 -> 217.8 mm
- net Button_X: track 69.8 -> 71.0 mm
- net Button_A: track 71.0 -> 69.8 mm
- net Button_Y: track 70.4 -> 71.0 mm
- net Button_B: track 71.0 -> 70.4 mm
