File: 07_Schémas/manette_2019/manette_2019.kicad_pcb (KiCad board)
At the start: 2 copper layers, 28 parts, among them J1 Power, SW1 Button_A, SW10 Button_DOWN, SW11 R_bumper, SW12 L_bumper, SW2 Button_B, SW3 Button_X, SW4 Button_Y, SW5 Button_START, SW6 Button_SELECT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

Commit message: update
Parts:
- removed SW11: R_bumper, Button_Switch_THT:Bouton_MEC
- removed SW12: L_bumper, Button_Switch_THT:Bouton_MEC
- added C1: C, Capacitor_THT:C_Disc_D5.0mm_W2.5mm_P5.00mm, F.Cu at (104.6, 102.1)
- added C2: C, Capacitor_THT:C_Disc_D5.0mm_W2.5mm_P5.00mm, F.Cu at (81.5, 77.7)
- added C3: C, Capacitor_THT:C_Disc_D5.0mm_W2.5mm_P5.00mm, F.Cu at (144.5, 78.7)
- added C4: C, Capacitor_THT:C_Disc_D5.0mm_W2.5mm_P5.00mm, F.Cu at (167.9, 116.3)
- added C5: C, Capacitor_THT:C_Disc_D5.0mm_W2.5mm_P5.00mm, F.Cu at (81.5, 69.6)
- added C6: C, Capacitor_THT:C_Disc_D5.0mm_W2.5mm_P5.00mm, F.Cu at (138.2, 91.7)
- added J2: Screw_Terminal_01x04, TerminalBlock:TerminalBlock_bornier-4_P5.08mm, F.Cu at (169.4, 51.8)
- added J3: Screw_Terminal_01x04, TerminalBlock:TerminalBlock_bornier-4_P5.08mm, F.Cu at (51.1, 50.8)
- added R4: R, Resistor_THT:R_Axial_DIN0309_L9.0mm_D3.2mm_P15.24mm_Horizontal, F.Cu at (144.5, 48.0)
- added SW13: Calib, Button_Switch_THT:Bouton_MEC, F.Cu at (127.5, 139.4)
- added U4: OLED_Display, OLED:OLED RGB, F.Cu at (121.4, 70.4)
- added U8: PCA9306, PCA9306:PCA9306, F.Cu at (57.4, 114.3)
- added Y1: Resonator, Crystal:Resonator-3Pin_W6.0mm_H3.0mm, F.Cu at (80.8, 90.4)
- JS1: value Joystick_RSF_2-Axis -> Joystick_Left
- JS2: value Joystick_RSF_2-Axis -> Joystick_Right
- moved SW9 151.8 mm to (61.0, 124.5)
- moved SW10 132.5 mm to (73.7, 137.2)
- moved SW8 129.1 mm to (73.7, 111.8)
- moved SW7 108.8 mm to (86.4, 124.5)
- moved LS1 108.6 mm to (54.6, 90.2), turned to 270 degrees
- moved U5 105.4 mm to (117.9, 136.1), turned to 270 degrees
- moved R3 92.9 mm to (71.1, 102.6), turned to 90 degrees
- moved SW5 90.0 mm to (129.5, 96.5)
- moved SW4 66.1 mm to (175.3, 63.5)
- moved U2 64.1 mm to (85.6, 63.0)
- moved D3 57.4 mm to (65.3, 97.5), turned to 90 degrees
- moved JS2 57.1 mm to (156.0, 118.9)
- moved U6 56.4 mm to (178.1, 126.0), turned to 180 degrees
- moved U3 55.7 mm to (155.7, 88.6), turned to 180 degrees
- moved D2 55.4 mm to (83.6, 50.8)
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Connections:
- D1 pad 2: +5V -> +3.3V
- D2 pad 2: +5V -> +3.3V
- D3 pad 1: +5V -> +3.3V
- J1 pad 2: Net-(J1-Pad2) -> +9V
- U1 pad 15: +10V -> +9V
- U2 pad 2: Net-(U2-Pad2) -> RX_Atmega
- U2 pad 3: Net-(U2-Pad3) -> TX_Atmega
- U2 pad 6: Net-(U2-Pad6) -> Calib
- U3 pad 18: +5V -> Net-(R4-Pad2)
- U3 pad 2: Calib -> Net-(U3-Pad2)
- U3 pad 9: Net-(U3-Pad9) -> +5V
- U6 pad 1: +10V -> +9V
- U7 pad 1: +10V -> +9V
Routing:
- net GND: track 0.00 -> 39.6 mm
- net +9V: track 0.00 -> 32.0 mm
Other:
- board outline added: 150 x 100 mm
- rule via_min_size: 0.4 -> 0.8

Commit message: update schema
Parts:
- removed U4: OLED_Display, OLED:OLED RGB
- added C7: C, Capacitor_THT:C_Rect_L7.0mm_W3.5mm_P5.00mm, F.Cu at (158.0, 57.0)
- added C8: C, Capacitor_THT:C_Rect_L7.0mm_W3.5mm_P5.00mm, F.Cu at (155.0, 65.1)
- added C9: C, Capacitor_THT:C_Radial_D10.0mm_H20.0mm_P5.00mm, F.Cu at (178.0, 136.7)
- added J4: OLED_Display, TerminalBlock_4Ucon:TerminalBlock_4Ucon_1x09_P3.50mm_Horizontal, F.Cu at (106.3, 50.8)
- C1, C2, C3, C4, C5, C6: footprint Capacitor_THT:C_Disc_D5.0mm_W2.5mm_P5.00mm -> Capacitor_THT:C_Rect_L7.0mm_W3.5mm_P5.00mm
- moved C5 78.3 mm to (158.0, 52.9), turned to 0 degrees
- moved C2 73.3 mm to (150.5, 52.9), turned to 0 degrees
- moved C4 61.8 mm to (150.5, 57.0), turned to 0 degrees
- moved U3 44.9 mm to (145.0, 132.2)
- moved U1 39.5 mm to (121.3, 79.6)
- moved C1 37.7 mm to (119.1, 67.3), turned to 0 degrees
- moved U2 36.5 mm to (96.6, 97.7)
- moved C6 35.0 mm to (155.0, 61.0)
- moved C3 27.4 mm to (150.3, 105.5)
- moved SW5 8.55 mm to (128.4, 105.0)
- moved SW6 8.47 mm to (114.7, 105.1)
- moved SW13 4.36 mm to (131.8, 139.9)
- moved U5 2.96 mm to (120.8, 136.2)
Connections:
- C1 pad 1: +9V -> VCC
- J1 pad 2: +9V -> VCC
- U1 pad 15: +9V -> Net-(U1-Pad15)
- U6 pad 1: +9V -> VCC
- U7 pad 1: +9V -> VCC
Routing:
- net VCC: track 0.00 -> 34.1 mm
- net +9V: track 32.0 -> 0.00 mm
- net GND: track 39.6 -> 41.1 mm

Commit message: Plans et data movement
Parts:
- removed C8: C, Capacitor_THT:C_Rect_L7.0mm_W3.5mm_P5.00mm
- removed C9: C, Capacitor_THT:C_Radial_D10.0mm_H20.0mm_P5.00mm
- removed D1: LED_B, LED_THT:LED_D3.0mm
- removed D2: LED_R, LED_THT:LED_D3.0mm
- removed R1, R2: R, Resistor_THT:R_Axial_DIN0309_L9.0mm_D3.2mm_P15.24mm_Horizontal
- removed SW1: Button_A, Button_Switch_THT:Bouton_MEC
- removed SW10: Button_DOWN, Button_Switch_THT:Bouton_MEC
- removed SW13: Calib, Button_Switch_THT:Bouton_MEC
- removed SW2: Button_B, Button_Switch_THT:Bouton_MEC
- removed SW3: Button_X, Button_Switch_THT:Bouton_MEC
- removed SW4: Button_Y, Button_Switch_THT:Bouton_MEC
- removed SW5: Button_START, Button_Switch_THT:Bouton_MEC
- removed SW6: Button_SELECT, Button_Switch_THT:Bouton_MEC
- removed SW7: Button_RIGHT, Button_Switch_THT:Bouton_MEC
- removed SW8: Button_UP, Button_Switch_THT:Bouton_MEC
- removed SW9: Button_LEFT, Button_Switch_THT:Bouton_MEC
- added D4: D, Diode_THT:D_A-405_P10.16mm_Horizontal, F.Cu at (95.2, 86.4)
- added J10: Alim_LED, TerminalBlock:TerminalBlock_bornier-2_P5.08mm, B.Cu at (132.1, 94.6)
- added J5: Rumble, TerminalBlock:TerminalBlock_bornier-2_P5.08mm, B.Cu at (105.4, 94.6)
- added J6: Calib, Connector_PinSocket_2.54mm:PinSocket_1x02_P2.54mm_Vertical, F.Cu at (87.6, 95.2)
- added J7: Conn_R_Button, manette_2019:Conn_8, F.Cu at (134.9, 55.9)
- added J8: Conn_L_Button, manette_2019:Conn_8, F.Cu at (8.64, 61.5)
- added J9: Conn_Middle_PCB, manette_2019:Conn_8, F.Cu at (75.8, 52.0)
- added R15: R, Resistor_THT:R_Axial_DIN0309_L9.0mm_D3.2mm_P15.24mm_Horizontal, F.Cu at (90.2, 90.2)
- added REF**: MountingHole_3.2mm_M3, MountingHole:MountingHole_3.2mm_M3, F.Cu at (8.00, 82.0)
- added REF**: MountingHole_3.2mm_M3, MountingHole:MountingHole_3.2mm_M3, F.Cu at (114.3, 81.3)
- added REF**: MountingHole_3.2mm_M3, MountingHole:MountingHole_3.2mm_M3, F.Cu at (73.7, 20.6)
- added RV1: R_POT, Potentiometer_THT:Potentiometer_Bourns_PTA2043_Single_Slide, B.Cu at (15.5, 3.75)
- added RV2: R_POT, Potentiometer_THT:Potentiometer_Bourns_PTA2043_Single_Slide, B.Cu at (131.0, 3.75)
- C1: footprint Capacitor_THT:C_Rect_L7.0mm_W3.5mm_P5.00mm -> Capacitor_THT:C_Radial_D10.0mm_H20.0mm_P5.00mm; moved to B.Cu
- J1: value Power -> Vcc; moved to B.Cu
- J2: value Screw_Terminal_01x04 -> L_Bumper; footprint TerminalBlock:TerminalBlock_bornier-4_P5.08mm -> Connector_PinSocket_2.54mm:PinSocket_1x02_P2.54mm_Vertical
- J3: value Screw_Terminal_01x04 -> R_Bumper; footprint TerminalBlock:TerminalBlock_bornier-4_P5.08mm -> Connector_PinSocket_2.54mm:PinSocket_1x02_P2.54mm_Vertical
- J4: footprint TerminalBlock_4Ucon:TerminalBlock_4Ucon_1x09_P3.50mm_Horizontal -> Connector_PinSocket_2.54mm:PinSocket_1x09_P2.54mm_Vertical
- LS1: moved to B.Cu
- U1: footprint ESP32:ESP32 -> manette_2019:ESP32
- U8: footprint PCA9306:PCA9306 -> manette_2019:PCA9306
- moved U3 135.8 mm to (89.5, 8.26), turned to 0 degrees
- moved C2 127.6 mm to (22.9, 51.4)
- moved J2 121.6 mm to (57.1, 5.00), turned to 270 degrees
- moved C6 114.6 mm to (43.1, 85.5), turned to 180 degrees
- moved U5 91.7 mm to (69.2, 60.3), turned to 0 degrees
- moved U1 83.3 mm to (38.7, 68.6)
- moved J1 82.5 mm to (120.0, 94.6), turned to 0 degrees
- moved C5 76.3 mm to (85.7, 28.6), turned to 270 degrees
- moved U6 76.3 mm to (125.1, 71.1), turned to 0 degrees
- moved JS2 74.2 mm to (105.0, 65.0), turned to 180 degrees
- moved J4 69.8 mm to (46.0, 15.7), turned to 90 degrees
- moved C7 66.3 mm to (92.1, 50.8)
- moved J3 63.5 mm to (94.0, 4.00), turned to 270 degrees
- moved LS1 61.0 mm to (76.9, 33.4)
- moved D3 58.1 mm to (71.2, 39.7)
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Connections:
- C2 pad 1: +5V -> VCC
- C3 pad 1: +5V -> VCC
- C4 pad 1: +5V -> VCC
- C6 pad 1: +3.3V -> +5V
- C7 pad 1: VCC -> +3.3V
- D3 pad 1: +3.3V -> VCC
- J1 pad 1: GND -> VCC
- J2 pad 1: Right_trigger -> L_Bumper
- J2 pad 2: R_Bumper -> GND
- J3 pad 1: Left_trigger -> R_Bumper
- J3 pad 2: L_Bumper -> GND
- LS1 pad 2: +3.3V -> VCC
- U1 pad 10: OLEDCS -> DC
- U1 pad 15: Net-(U1-Pad15) -> VCC
- U1 pad 24: Connected -> Rumble
- U1 pad 25: Power -> Buzzer
- U1 pad 26: Buzzer -> Connected
- U1 pad 8: RESET -> OLEDCS
- U1 pad 9: DC -> RESET
- U3 pad 1: Net-(U3-Pad1) -> L_Bumper
- U3 pad 2: Net-(U3-Pad2) -> Left_joystick_button
- U3 pad 21: Button_SELECT -> Net-(U3-Pad21)
- U3 pad 22: Button_START -> Net-(U3-Pad22)
- U3 pad 23: L_Bumper -> Right_joystick_button
- U3 pad 24: R_Bumper -> Button_A
- U3 pad 25: Button_X -> Button_B
- U3 pad 27: Button_B -> Button_X
- U3 pad 28: Button_A -> R_Bumper
- U3 pad 3: R_joystick_button -> Button_DOWN
- U3 pad 4: L_joystick_button -> Button_RIGHT
- U3 pad 5: Button_LEFT -> Button_UP
- U3 pad 6: Button_UP -> Button_LEFT
- U3 pad 7: Button_RIGHT -> Button_SELECT
- U3 pad 8: Button_DOWN -> Button_START
- U5 pad 1: Connected -> Rumble
- U5 pad 16: Net-(R3-Pad1) -> Conn_LED_On
- U5 pad 17: Net-(R2-Pad1) -> Net-(R3-Pad1)
- U5 pad 2: Power -> Buzzer
- U5 pad 3: Buzzer -> Connected
- U8 pad 2: RX_Atmega -> TX_Atmega
- U8 pad 3: TX_Atmega -> RX_Atmega
- U8 pad 6: RX_ESP32 -> TX_ESP32
- U8 pad 7: TX_ESP32 -> RX_ESP32
Routing:
- net GND: track 41.1 -> 754.7 mm
- net +5V: track 0.00 -> 579.6 mm
- net R_trigger: track 0.00 -> 248.1 mm
- net VCC: track 34.1 -> 267.3 mm
- net VCC_LED: track 0.00 -> 217.8 mm
- net L_trigger: track 0.00 -> 152.4 mm
- net +3.3V: track 0.00 -> 149.4 mm
- net Button_LEFT: track 0.00 -> 118.4 mm
- net Button_UP: track 0.00 -> 117.0 mm
- net Button_RIGHT: track 0.00 -> 115.3 mm
- net Button_DOWN: track 0.00 -> 113.8 mm
- net SCL: track 0.00 -> 103.4 mm
- net SDA: track 0.00 -> 100.9 mm
- net MISO: track 0.00 -> 75.0 mm
- net Button_Y: track 0.00 -> 71.0 mm
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- added copper zone on F.Cu, net GND
- added copper zone on B.Cu, net VCC
Other:
- outline, holes or cut-outs redrawn
- net class Default: trace_width 0.25 -> 0.5

Commit message: update
Routing:
- net Left_joystick_button: track 53.7 -> 54.3 mm
Changed lines of the file:
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@@
   (segment (start 87.63 97.155) (end 86.995 97.79) (width 0.5) (layer F.Cu) (net 16))
   (segment (start 87.63 10.795) (end 89.535 10.795) (width 0.5) (layer F.Cu) (net 18))
-  (segment (start 48.25 27.1) (end 49.95 25.4) (width 0.5) (layer F.Cu) (net 18))
-  (segment (start 48.25 28.05) (end 48.25 27.1) (width 0.5) (layer F.Cu) (net 18))
-  (segment (start 49.95 25.4) (end 81.026 25.4) (width 0.5) (layer F.Cu) (net 18))
+  (segment (start 48.25 26.045) (end 48.895 25.4) (width 0.5) (layer F.Cu) (net 18))
+  (segment (start 48.25 28.05) (end 48.25 26.045) (width 0.5) (layer F.Cu) (net 18))
+  (segment (start 48.895 25.4) (end 81.026 25.4) (width 0.5) (layer F.Cu) (net 18))
+  (segment (start 81.026 25.4) (end 83.82 22.606) (width 0.5) (layer F.Cu) (net 18))
   (segment (start 83.82 22.606) (end 83.82 14.605) (width 0.5) (layer F.Cu) (net 18))
-  (segment (start 81.026 25.4) (end 83.82 22.606) (width 0.5) (layer F.Cu) (net 18))
   (segment (start 83.82 14.605) (end 87.63 10.795) (width 0.5) (layer F.Cu) (net 18))
   (segment (start 108.25 52.1) (end 107.315 51.165) (width 0.5) (layer B.Cu) (net 25))

Commit message: update
Parts:
- removed C3, C4: C, Capacitor_THT:C_Rect_L7.0mm_W3.5mm_P5.00mm
- removed U6: R-783.3-0.5, Converter_DCDC:Converter_DCDC_RECOM_R-78E-0.5_THT
- removed U7: R-78E5.0-0.5, Converter_DCDC:Converter_DCDC_RECOM_R-78E-0.5_THT
- moved C7 41.8 mm to (63.8, 20.0)
- moved REF** 4.03 mm to (77.7, 20.6)
Connections:
- C1 pad 1: VCC -> +5V
- C2 pad 1: VCC -> +5V
- C7 pad 1: +3.3V -> +5V
- D3 pad 1: VCC -> +5V
- D4 pad 1: VCC -> +5V
- J1 pad 1: VCC -> +5V
- J1 pad 2: VCC -> +5V
- J4 pad 8: +3.3V -> +5V
- J5 pad 2: VCC -> +5V
- J7 pad 2: Button_A -> Button_Y
- J7 pad 6: Button_Y -> Button_A
- J8 pad 2: Button_DOWN -> Button_UP
- J8 pad 6: Button_UP -> Button_DOWN
- J9 pad 6: VCC -> +5V
- LS1 pad 2: VCC -> +5V
- U1 pad 15: VCC -> +5V
- U1 pad 16: Net-(U1-Pad16) -> +3.3V
- U3 pad 24: Button_A -> Button_Y
- U3 pad 26: Button_Y -> Button_A
- U3 pad 3: Button_DOWN -> Button_UP
- U3 pad 5: Button_UP -> Button_DOWN
Routing:
- net VCC: track 267.3 -> 0.00 mm
- net +3.3V: track 149.4 -> 58.3 mm
- net R_trigger: track 248.1 -> 195.2 mm
- net MISO: track 75.0 -> 119.9 mm
- net +5V: track 579.6 -> 555.7 mm
- net SDCS: track 49.7 -> 68.6 mm
- net GND: track 754.7 -> 747.9 mm
- net OLEDCS: track 60.6 -> 65.7 mm
- net Button_X: track 71.0 -> 66.9 mm
- net Button_Y: track 71.0 -> 67.1 mm
- net Button_UP: track 117.0 -> 113.2 mm
- net DC: track 56.0 -> 59.8 mm
- net RESET: track 58.2 -> 62.0 mm
- net Button_B: track 70.4 -> 66.9 mm
- net SCK: track 53.4 -> 56.5 mm
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- added copper zone on B.Cu, net +5V
- removed copper zone on B.Cu, net VCC
Other:
- board text added: "P1704 Manette Intelligence MCT 2018-2019 AKC"

Commit message: update
Parts:
- C1, LS1: moved to F.Cu
- RV1: value R_POT -> L_POT; footprint Potentiometer_THT:Potentiometer_Bourns_PTA2043_Single_Slide -> manette_2019:Potentiomètre linéaire
- RV2: footprint Potentiometer_THT:Potentiometer_Bourns_PTA2043_Single_Slide -> manette_2019:Potentiomètre linéaire
- moved RV1 16.4 mm to (17.5, 20.0), turned to 180 degrees
- moved RV2 16.3 mm to (132.5, 20.0), turned to 180 degrees
- moved REF** 9.45 mm to (7.62, 91.4)
- moved D3 7.07 mm to (64.1, 39.7)
- moved J8 6.86 mm to (8.64, 54.6)
- moved R3 6.44 mm to (59.1, 44.8)
- moved R4 3.81 mm to (104.8, 48.9)
- moved U3 3.81 mm to (93.3, 8.26)
- moved C5 3.18 mm to (88.9, 28.6)
- moved REF** 1.49 mm to (76.2, 20.6)
- moved LS1 0.09 mm to (76.8, 33.4)
- turned J7 to 270 degrees
- turned J9 to 0 degrees
Connections:
- U1 pad 1: Net-(U1-Pad1) -> +3.3V
- U1 pad 10: DC -> Buzzer
- U1 pad 11: SCK -> Connected
- U1 pad 12: MISO -> RX_ESP32
- U1 pad 13: MOSI -> TX_ESP32
- U1 pad 14: GND -> Net-(U1-Pad14)
- U1 pad 15: +5V -> Net-(U1-Pad15)
- U1 pad 16: +3.3V -> Net-(U1-Pad16)
- U1 pad 22: Net-(U1-Pad22) -> SDCS
- U1 pad 23: Net-(U1-Pad23) -> OLEDCS
- U1 pad 24: Rumble -> RESET
- U1 pad 25: Buzzer -> DC
- U1 pad 26: Connected -> SCK
- U1 pad 27: RX_ESP32 -> MISO
- U1 pad 28: TX_ESP32 -> MOSI
- U1 pad 29: Net-(U1-Pad29) -> GND
- U1 pad 30: Net-(U1-Pad30) -> +5V
- U1 pad 7: SDCS -> Net-(U1-Pad7)
- U1 pad 8: OLEDCS -> Net-(U1-Pad8)
- U1 pad 9: RESET -> Rumble
Routing:
- net GND: track 747.9 -> 700.2 mm
- net Button_SELECT: track 38.4 -> 65.8 mm
- net Button_X: track 66.9 -> 88.8 mm
- net Button_START: track 35.8 -> 54.3 mm
- net Button_A: track 66.9 -> 82.8 mm
- net SCL: track 103.4 -> 115.1 mm
- net Button_B: track 66.9 -> 75.7 mm
- net Conn_LED_On: track 17.8 -> 25.7 mm
- net SDA: track 100.9 -> 108.7 mm
- net VCC_LED: track 214.8 -> 222.1 mm
- net Net-(D3-Pad2): track 11.4 -> 17.9 mm
- net Net-(R3-Pad1): track 23.9 -> 30.1 mm
- net Connected: track 34.0 -> 28.7 mm
- net Button_UP: track 113.2 -> 118.2 mm
- net Buzzer: track 37.5 -> 32.6 mm
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Other:
- outline, holes or cut-outs redrawn

Commit message: update
Parts:
- moved JS1 10.0 mm to (35.0, 40.0)
- moved JS2 10.0 mm to (115.0, 65.0)
Connections:
- JS1 pad 2: Left_joystick_analog_x -> L_joystick_analog_x
- JS1 pad 5: Left_joystick_analog_y -> L_joystick_analog_y
- JS2 pad 2: Right_joystick_analog_x -> R_joystick_analog_x
- JS2 pad 5: Right_joystick_analog_y -> R_joystick_analog_y
Routing:
- net GND: track 700.2 -> 621.9 mm
- net MISO: track 118.8 -> 72.1 mm
- net SCK: track 60.3 -> 19.2 mm
- net DC: track 62.3 -> 22.3 mm
- net RESET: track 63.4 -> 24.3 mm
- net SDCS: track 68.1 -> 29.0 mm
- net OLEDCS: track 66.1 -> 27.0 mm
- net MOSI: track 58.3 -> 21.6 mm
- net +5V: track 555.3 -> 531.6 mm
- net Right_joystick_button: track 36.6 -> 40.7 mm
- net Left_joystick_button: track 58.1 -> 56.1 mm
- net Net-(R15-Pad1): track 42.4 -> 40.6 mm
- net L_trigger: track 145.9 -> 147.1 mm

Commit message: update
Parts:
- removed the REF** at (114.3, 81.3)
- removed the REF** at (76.2, 20.6)
- added REF**: MountingHole_3.2mm_M3, MountingHole:MountingHole_3.2mm_M3, F.Cu at (132.8, 114.0)
- added REF**: MountingHole_3.2mm_M3, MountingHole:MountingHole_3.2mm_M3, F.Cu at (-95.9, 56.8)
- moved J10 124.8 mm to (10.7, 65.5), turned to 270 degrees
- moved J1 118.0 mm to (10.7, 50.3), turned to 270 degrees
- moved C1 110.1 mm to (18.3, 55.9), turned to 270 degrees
- moved R3 74.4 mm to (125.0, 79.2), turned to 270 degrees
- moved D3 72.2 mm to (120.9, 84.3), turned to 270 degrees
- moved LS1 63.9 mm to (110.2, 87.9), turned to 90 degrees
- moved J8 62.8 mm to (71.1, 60.5)
- moved U5 62.7 mm to (131.6, 53.8)
- moved R15 57.5 mm to (147.6, 87.0), turned to 180 degrees
- moved U1 55.4 mm to (80.6, 32.4)
- moved REF** 53.7 mm to (-37.6, 120.4)
- moved C2 53.5 mm to (62.2, 15.2)
- moved U2 49.0 mm to (6.22, 89.2), turned to 90 degrees
- moved D4 47.4 mm to (142.5, 83.2), turned to 180 degrees
- moved C5 46.0 mm to (74.2, 72.1)
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Connections:
- J7 pad 2: Button_Y -> Button_A
- J7 pad 4: Button_B -> Button_X
- J7 pad 6: Button_A -> Button_Y
- J7 pad 8: Button_X -> Button_B
- U2 pad 25: L_joystick_analog_x -> L_joystick_analog_y
- U2 pad 26: L_joystick_analog_y -> L_joystick_analog_x
- U3 pad 24: Button_Y -> Button_A
- U3 pad 25: Button_B -> Button_X
- U3 pad 26: Button_A -> Button_Y
- U3 pad 27: Button_X -> Button_B
- U3 pad 7: Button_SELECT -> Button_START
- U3 pad 8: Button_START -> Button_SELECT
Routing:
- net R_joystick_analog_y: track 0.00 -> 157.8 mm
- net R_joystick_analog_x: track 0.00 -> 156.3 mm
- net Conn_LED_On: track 25.7 -> 143.1 mm
- net Button_LEFT: track 121.8 -> 7.47 mm
- net Button_DOWN: track 120.0 -> 7.47 mm
- net Button_RIGHT: track 118.8 -> 7.47 mm
- net Button_UP: track 118.2 -> 7.47 mm
- net R_Bumper: track 9.84 -> 104.6 mm
- net GND: track 621.9 -> 529.6 mm
- net VCC_LED: track 222.1 -> 133.2 mm
- net Button_X: track 88.8 -> 6.46 mm
- net Button_A: track 82.8 -> 6.46 mm
- net Button_B: track 75.7 -> 6.46 mm
- net TX_ESP32: track 31.2 -> 96.9 mm
- net L_trigger: track 147.1 -> 83.9 mm
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- removed copper zone on B.Cu, net +5V
- removed copper zone on F.Cu, net GND
