File: 07_Schémas/manette_2019/manette_2019.kicad_pcb (KiCad board)
At the start: 2 copper layers, 150 x 100 mm, 34 parts, among them J1 Vcc, J10 Alim_LED, J2 L_Bumper, J3 R_Bumper, J4 OLED_Display, J5 Rumble, J6 Calib, J7 Conn_R_Button, J8 Conn_L_Button, J9 Conn_Middle_PCB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

Commit message: update
Parts:
- removed the REF** at (-37.6, 120.4)
- removed the REF** at (132.8, 114.0)
- removed the REF** at (-95.9, 56.8)
- added REF**: MountingHole_3.2mm_M3, MountingHole:MountingHole_3.2mm_M3, F.Cu at (96.5, 12.1)
- added REF**: MountingHole_3.2mm_M3, MountingHole:MountingHole_3.2mm_M3, F.Cu at (144.8, 95.9)
- added REF**: MountingHole_3.2mm_M3, MountingHole:MountingHole_3.2mm_M3, F.Cu at (5.08, 95.9)
- U8: moved to B.Cu
- moved U8 16.0 mm to (41.9, 64.8)
- moved J4 3.17 mm to (69.8, 10.2)
- moved U2 3.12 mm to (7.62, 86.4)
- moved J6 3.06 mm to (60.3, 92.7)
- moved Y1 2.64 mm to (31.7, 91.4)
- moved C6 2.54 mm to (18.3, 91.4)
- moved C7 1.78 mm to (85.1, 5.08)
- moved J3 1.78 mm to (102.4, 5.08)
- moved J1 1.78 mm to (10.7, 52.1)
- moved J2 1.19 mm to (56.7, 5.08)
Routing:
- net TX_ESP32: track 96.9 -> 67.8 mm
- net RX_ESP32: track 82.8 -> 58.7 mm
- net +5V: track 552.3 -> 538.1 mm
- net +3.3V: track 37.0 -> 23.9 mm
- net L_joystick_analog_y: track 50.1 -> 40.2 mm
- net GND: track 529.6 -> 536.7 mm
- net RX_Atmega: track 49.6 -> 44.8 mm
- net Calib: track 46.7 -> 50.6 mm
- net L_joystick_analog_x: track 53.2 -> 49.8 mm
- net VCC_LED: track 133.2 -> 129.9 mm
- net RESET: track 13.7 -> 10.5 mm
- net OLEDCS: track 13.7 -> 10.5 mm
- net MOSI: track 12.7 -> 9.53 mm
- net SDCS: track 13.7 -> 10.5 mm
- net SCK: track 13.7 -> 10.5 mm
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- added copper zone on B.Cu, net +5V
- added copper zone on F.Cu, net GND

Commit message: update
Parts:
- moved REF** 21.2 mm to (76.2, 6.10)
- moved J4 3.70 mm to (71.8, 13.3)
- moved REF** 1.91 mm to (144.8, 94.0)
- moved REF** 1.73 mm to (6.10, 94.5)
Connections:
- U2 pad 20: Net-(U2-Pad20) -> +5V
Routing:
- net +5V: track 538.1 -> 574.5 mm
- net GND: track 536.7 -> 547.4 mm
- net MISO: track 60.5 -> 54.5 mm
- net OLEDCS: track 10.5 -> 6.51 mm
- net SDCS: track 10.5 -> 6.51 mm
- net SCK: track 10.5 -> 6.51 mm
- net RESET: track 10.5 -> 6.51 mm
- net DC: track 10.5 -> 6.51 mm
- net MOSI: track 9.53 -> 7.14 mm
- net R_joystick_analog_y: track 155.6 -> 154.4 mm
- net R_joystick_analog_x: track 155.5 -> 154.7 mm
- net Conn_LED_On: track 143.1 -> 142.5 mm

Commit message: update
Parts:
- added R1: R, Resistor_THT:R_Axial_DIN0309_L9.0mm_D3.2mm_P15.24mm_Horizontal, F.Cu at (55.6, 88.9)
- added R2: R, Resistor_THT:R_Axial_DIN0309_L9.0mm_D3.2mm_P15.24mm_Horizontal, F.Cu at (55.6, 84.1)
- moved C2 55.5 mm to (105.9, 49.5), turned to 180 degrees
- moved J4 8.83 mm to (80.6, 13.1)
- moved C7 6.97 mm to (90.9, 8.89)
- moved U1 6.73 mm to (87.4, 32.3), turned to 90 degrees
Connections:
- U1 pad 10: Buzzer -> MISO
- U1 pad 11: Connected -> Net-(U1-Pad11)
- U1 pad 12: RX_ESP32 -> Net-(U1-Pad12)
- U1 pad 13: TX_ESP32 -> Net-(U1-Pad13)
- U1 pad 15: Net-(U1-Pad15) -> MOSI
- U1 pad 22: SDCS -> Rumble
- U1 pad 23: OLEDCS -> Buzzer
- U1 pad 24: RESET -> Connected
- U1 pad 25: DC -> Net-(U1-Pad25)
- U1 pad 26: SCK -> Net-(U1-Pad26)
- U1 pad 27: MISO -> Net-(U1-Pad27)
- U1 pad 28: MOSI -> Net-(U1-Pad28)
- U1 pad 3: Net-(U1-Pad3) -> SDCS
- U1 pad 4: Net-(U1-Pad4) -> OLEDCS
- U1 pad 5: Net-(U1-Pad5) -> RESET
- U1 pad 6: Net-(U1-Pad6) -> RX_ESP32
- U1 pad 7: Net-(U1-Pad7) -> TX_ESP32
- U1 pad 8: Net-(U1-Pad8) -> DC
- U1 pad 9: Rumble -> SCK
Routing:
- net +3.3V: track 23.9 -> 108.4 mm
- net L_Bumper: track 67.0 -> 143.2 mm
- net +5V: track 574.5 -> 624.9 mm
- net RX_ESP32: track 58.7 -> 96.3 mm
- net TX_ESP32: track 67.8 -> 96.3 mm
- net MISO: track 54.5 -> 44.2 mm
- net MOSI: track 7.14 -> 16.5 mm
- net Rumble: track 78.2 -> 84.8 mm
- net R_Bumper: track 102.8 -> 107.7 mm
- net Connected: track 84.6 -> 79.8 mm
- net RESET: track 6.51 -> 9.84 mm
- net SDCS: track 6.51 -> 9.54 mm
- net OLEDCS: track 6.51 -> 9.22 mm
- net GND: track 547.4 -> 549.6 mm
- net Left_joystick_button: track 59.2 -> 57.5 mm
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