File: 07_Schémas/PCB_test_NKK/PCB_test_NKK.kicad_pcb (KiCad board)
At the start: 2 copper layers, 3 parts, among them J1 Conn_01x05, J2 Conn_01x05, U1 NKK_Smartswitch

Commit message: update
Parts:
- added C1: C, Capacitor_THT:C_Rect_L7.2mm_W3.5mm_P5.00mm_FKS2_FKP2_MKS2_MKP2, F.Cu at (76.8, 82.5)
- added C2: C, Capacitor_THT:CP_Radial_D10.0mm_P5.00mm, F.Cu at (76.8, 90.8)
- added J3: Conn_01x03, TerminalBlock_Phoenix:TerminalBlock_Phoenix_MPT-0,5-3-2.54_1x03_P2.54mm_Horizontal, F.Cu at (102.2, 101.0)
- added J4: Conn_01x02, TerminalBlock_Phoenix:TerminalBlock_Phoenix_MPT-0,5-2-2.54_1x02_P2.54mm_Horizontal, F.Cu at (76.8, 101.0)
- added U2: NKK_Smartswitch, NKK:NKK_Switch, F.Cu at (101.0, 43.2)
- added U3: R-783.3-0.5, Converter_DCDC:Converter_DCDC_RECOM_R-78E-0.5_THT, F.Cu at (76.8, 75.6)
- J1, J2: value Conn_01x05 -> Conn_01x03; footprint NKK:conn_01x05 -> TerminalBlock_Phoenix:TerminalBlock_Phoenix_MPT-0,5-3-2.54_1x03_P2.54mm_Horizontal
- moved J1 56.0 mm to (92.7, 101.0), turned to 0 degrees
- moved U1 33.0 mm to (101.0, 69.8), turned to 180 degrees
- moved J2 32.8 mm to (83.8, 101.0), turned to 0 degrees
Connections:
- net Net-(J2-Pad3) renamed DC1
- J1 pad 1: Net-(J1-Pad1) -> SDI
- J1 pad 2: Net-(J1-Pad2) -> SCK
- J1 pad 3: Net-(J1-Pad3) -> Rst
- J2 pad 1: Net-(J2-Pad1) -> SW1
- J2 pad 2: Net-(J2-Pad2) -> SS1
- U1 pad 1: Net-(J1-Pad5) -> SW1
- U1 pad 10: Net-(J1-Pad1) -> GND
- U1 pad 2: Net-(J1-Pad4) -> GND
- U1 pad 3: Net-(J1-Pad3) -> +3.3V
- U1 pad 4: Net-(J2-Pad1) -> SS1
- U1 pad 5: Net-(J2-Pad2) -> Rst
- U1 pad 7: Net-(J2-Pad4) -> SCK
- U1 pad 8: Net-(J2-Pad5) -> SDI
- U1 pad 9: Net-(J1-Pad2) -> +16V
Routing:
- net GND: track 0.00 -> 27.4 mm
- net +16V: track 0.00 -> 25.4 mm

Commit message: update schéma
Parts:
- moved U2 68.9 mm to (168.0, 58.9), turned to 90 degrees
- moved C1 62.9 mm to (135.6, 60.2)
- moved C2 62.9 mm to (135.6, 68.4)
- moved J4 62.9 mm to (135.6, 78.6)
- moved U3 62.5 mm to (135.7, 54.4)
- moved J3 53.6 mm to (150.9, 78.6)
- moved J1 39.7 mm to (125.5, 78.6)
- moved J2 36.0 mm to (112.2, 78.7)
- moved U1 30.6 mm to (129.7, 59.3), turned to 90 degrees
Connections:
- J3 pad 1: SW2 -> SS2
- J3 pad 3: SS2 -> SW2
Routing:
- net SDI: track 0.00 -> 97.0 mm
- net +16V: track 25.4 -> 97.7 mm
- net +3.3V: track 0.00 -> 71.6 mm
- net GND: track 27.4 -> 95.0 mm
- net SCK: track 0.00 -> 53.1 mm
- net Rst: track 0.00 -> 50.5 mm
- net SW1: track 0.00 -> 43.3 mm
- net SW2: track 0.00 -> 38.5 mm
- net DC2: track 0.00 -> 33.8 mm
- net DC1: track 0.00 -> 29.7 mm
- net SS2: track 0.00 -> 25.2 mm
- net SS1: track 0.00 -> 23.6 mm

Commit message: update
Parts:
- moved J3 7.64 mm to (143.3, 78.6)
- moved J2 3.67 mm to (115.8, 78.7)
Routing:
- net SDI: track 97.0 -> 79.2 mm
- net SW1: track 43.3 -> 33.0 mm
- net SW2: track 38.5 -> 47.2 mm
- net DC2: track 33.8 -> 41.2 mm
- net SS2: track 25.2 -> 32.4 mm
- net SS1: track 23.6 -> 18.4 mm
- net +16V: track 97.7 -> 92.7 mm
- net DC1: track 29.7 -> 25.2 mm
- net Rst: track 50.5 -> 54.0 mm
- net SCK: track 53.1 -> 54.4 mm
Other:
- board outline added: 66 x 38.1 mm

Commit message: finished pcb_nkk
Parts:
- added ?: MountingHole_3.2mm_M3, MountingHole:MountingHole_3.2mm_M3, F.Cu at (171.4, 47.0)
- added ?: MountingHole_3.2mm_M3, MountingHole:MountingHole_3.2mm_M3, F.Cu at (172.7, 88.2)
- added ?: MountingHole_3.2mm_M3, MountingHole:MountingHole_3.2mm_M3, F.Cu at (104.8, 47.0)
- added ?: MountingHole_3.2mm_M3, MountingHole:MountingHole_3.2mm_M3, F.Cu at (104.1, 88.2)
- moved J3 3.37 mm to (143.5, 81.9)
- moved J1 3.36 mm to (125.5, 81.9)
- moved J4 3.32 mm to (135.6, 81.9)
- moved J2 3.18 mm to (115.8, 81.9)
Routing:
- net GND: track 95.0 -> 147.8 mm
- net +16V: track 92.7 -> 73.9 mm
- net DC1: track 25.2 -> 30.3 mm, vias 0 -> 1
- net SS1: track 18.4 -> 23.2 mm, vias 0 -> 1
- net SW1: track 33.0 -> 37.6 mm
- net SCK: track 54.4 -> 58.8 mm, vias 0 -> 2
- net SDI: track 79.2 -> 83.5 mm
- net +3.3V: track 71.6 -> 67.4 mm
- net Rst: track 54.0 -> 58.3 mm, vias 0 -> 2
- net SS2: track 32.4 -> 35.1 mm
- net DC2: track 41.2 -> 43.8 mm
- net SW2: track 47.2 -> 49.8 mm
- added copper zone on F.Cu, net +16V
- added copper zone on B.Cu, net +3.3V
- added copper zone on B.Cu, net GND
Other:
- board size 66 x 38.1 mm -> 73.7 x 43.2 mm
- board text added: "+16V"
- board text added: "DC1"
- board text added: "DC2"
- board text added: "GND"
- board text added: "P1704 Manette NKK version 1.0 MCT 2018-2019 AKC"
- board text added: "Rst"
- board text added: "SCK"
- board text added: "SDI"
- board text added: "SS1"
- board text added: "SS2"
- board text added: "SW1"
- board text added: "SW2"
