File: 07_Schémas/Manette_2019_PCB_Central/Manette_2019_PCB_Central.kicad_pcb (KiCad board)
At the start: 2 copper layers, 35.6 x 27.9 mm, 9 parts, among them J1 Button_OUT, J2 Button_In, SW1 Button_Start, SW2 Button_Select

Commit message: update schema
Connections:
- net Alim_Button_Start_Select renamed Conn_LED_On
Changed lines of the file:
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@@
   (net 5 "Net-(R2-Pad2)")
   (net 6 Vcc)
-  (net 7 Alim_Button_Start_Select)
+  (net 7 Conn_LED_On)
   (net_class Default "Ceci est la Netclass par défaut."
     (clearance 0.2)
@@
     (uvia_dia 0.3)
     (uvia_drill 0.1)
-    (add_net Alim_Button_Start_Select)
+    (add_net Conn_LED_On)
     (add_net GND)
     (add_net "Net-(R1-Pad2)")
@@
     (pad "" np_thru_hole circle (at 0 2.54) (size 1.1 1.1) (drill 1.1) (layers *.Cu *.Mask))
     (pad 2 thru_hole circle (at 2.54 0) (size 2.2 2.2) (drill 1.1) (layers *.Cu *.Mask)
-      (net 7 Alim_Button_Start_Select))
+      (net 7 Conn_LED_On))
     (pad "" np_thru_hole circle (at 2.54 2.54) (size 1.1 1.1) (drill 1.1) (layers *.Cu *.Mask))
     (model ${KISYS3DMOD}/TerminalBlock_Phoenix.3dshapes/TerminalBlock_Phoenix_MPT-0,5-2-2.54_1x02_P2.54mm_Horizontal.wrl
@@
       (net 5 "Net-(R2-Pad2)"))
     (pad 2 thru_hole circle (at -5.08 -3.81) (size 2 2) (drill 0.8) (layers *.Cu *.Mask)
-      (net 7 Alim_Button_Start_Select))
+      (net 7 Conn_LED_On))
     (pad 1 thru_hole circle (at 5.08 -3.81) (size 2 2) (drill 0.8) (layers *.Cu *.Mask)
       (net 3 GND))

Commit message: update schema
Parts:
- removed J2: Button_In, TerminalBlock_Phoenix:TerminalBlock_Phoenix_MPT-0,5-3-2.54_1x03_P2.54mm_Horizontal
- J1: value Button_OUT -> Conn_Middle_PCB; footprint TerminalBlock_Phoenix:TerminalBlock_Phoenix_MPT-0,5-2-2.54_1x02_P2.54mm_Horizontal -> manette_2019:Conn_8; moved to B.Cu
- moved J1 3.02 mm to (125.3, 121.2), turned to 180 degrees
- moved REF** 1.02 mm to (111.6, 122.2)
Connections:
- J1 pad 1: Vcc -> button_SELECT
Routing:
- net button_SELECT: track 18.8 -> 32.6 mm
- net Conn_LED_On: track 42.5 -> 39.1 mm
- net Vcc: track 10.4 -> 8.23 mm
- net GND: track 60.2 -> 61.6 mm
Other:
- board size 35.6 x 27.9 mm -> 35.3 x 26.4 mm
- net class Default: trace_width 0.25 -> 0.5

Commit message: update
Parts:
- J1: moved to F.Cu
- moved REF** 1.83 mm to (125.5, 102.6)
- turned J1 to 0 degrees
Routing:
- net GND: track 61.6 -> 40.1 mm
- net button_SELECT: track 32.6 -> 21.2 mm
- net Conn_LED_On: track 39.1 -> 27.9 mm
- net button_START: track 20.4 -> 25.0 mm
Other:
- board size 35.3 x 26.4 mm -> 34.9 x 26 mm
