File: 07_Schémas/manette_2019_boutons/manette_2019_boutons.sch (KiCad schematic (older format))
At the start: 10 parts, among them J1 Conn_bouton_1, J2 Conn_bouton_2, SW1 Bouton_1, SW2 Bouton_2, SW3 Bouton_3, SW4 Bouton_4

Commit message: update schema
Connections:
- net labels added: Vcc_LED
- net labels removed: VCC
Other:
- note added: "Ce PCB sera produit en 2 exemplaires par manette,\nl'un d'eux comportera les boutons A B X et Y, alors\nque l'autre aura le pad directionnel.\n"
Changed lines of the file:
@@
 EESchema Schematic File Version 4
+LIBS:manette_2019_boutons-cache
 EELAYER 26 0
 EELAYER END
@@
 	4525 2200 4525 2300
 Text GLabel 3375 2800 2    50   Output ~ 0
-VCC
+Vcc_LED
 Text GLabel 3375 2700 2    50   Output ~ 0
 GND
@@
 Connection ~ 4525 3375
 Text GLabel 5325 3375 2    50   Input ~ 0
-VCC
+Vcc_LED
 Text GLabel 5325 2850 2    50   Input ~ 0
-VCC
+Vcc_LED
 Text GLabel 5325 2300 2    50   Input ~ 0
-VCC
+Vcc_LED
 Text GLabel 5325 1775 2    50   Input ~ 0
-VCC
+Vcc_LED
 Text GLabel 5025 1675 2    50   Output ~ 0
 Bouton_1
@@
 	-1   0    0    1
 $EndComp
+Text Notes 5975 2300 0    50   ~ 0
+Ce PCB sera produit en 2 exemplaires par manette,\nl'un d'eux comportera les boutons A B X et Y, alors\nque l'autre aura le pad directionnel.\n
 $EndSCHEMATC

Commit message: update schema
Parts:
- removed J2: Conn_bouton_2, TerminalBlock_Phoenix:TerminalBlock_Phoenix_MPT-0,5-3-2.54_1x03_P2.54mm_Horizontal, symbol Connector:Screw_Terminal_01x03
- J1: value Conn_bouton_1 -> Conn_bouton; footprint TerminalBlock_Phoenix:TerminalBlock_Phoenix_MPT-0,5-3-2.54_1x03_P2.54mm_Horizontal -> manette_2019:Conn_8; symbol Connector:Screw_Terminal_01x03 -> Connector_Generic:Conn_01x08
Changed lines of the file:
@@
 Text GLabel 3375 2800 2    50   Output ~ 0
 Vcc_LED
-Text GLabel 3375 2700 2    50   Output ~ 0
+Text GLabel 3375 2600 2    50   Output ~ 0
 GND
-Text GLabel 3375 2600 2    50   Input ~ 0
+Text GLabel 3375 2100 2    50   Input ~ 0
 Bouton_1
+Text GLabel 3375 2300 2    50   Input ~ 0
+Bouton_2
 Text GLabel 3375 2500 2    50   Input ~ 0
-Bouton_2
-Text GLabel 3375 2400 2    50   Input ~ 0
 Bouton_3
-Text GLabel 3375 2300 2    50   Input ~ 0
+Text GLabel 3375 2700 2    50   Input ~ 0
 Bouton_4
 $Comp
@@
 Bouton_4
 $Comp
-L Connector:Screw_Terminal_01x03 J1
+L Connector_Generic:Conn_01x08 J1
 U 1 1 5CC930DA
-P 3175 2700
-F 0 "J1" H 3300 2650 50  0000 C CNN
-F 1 "Conn_bouton_1" H 3525 2725 50  0000 C CNN
-F 2 "TerminalBlock_Phoenix:TerminalBlock_Phoenix_MPT-0,5-3-2.54_1x03_P2.54mm_Horizontal" H 3175 2700 50  0001 C CNN
-F 3 "~" H 3175 2700 50  0001 C CNN
-	1    3175 2700
+P 3175 2500
+F 0 "J1" H 3300 2450 50  0000 C CNN
+F 1 "Conn_bouton" H 3525 2525 50  0000 C CNN
+F 2 "manette_2019:Conn_8" H 3175 2500 50  0001 C CNN
+F 3 "~" H 3175 2500 50  0001 C CNN
+	1    3175 2500
 	-1   0    0    1
 $EndComp
-$Comp
-L Connector:Screw_Terminal_01x03 J2
-U 1 1 5CC93321
-P 3175 2400
-F 0 "J2" H 3300 2350 50  0000 C CNN
-F 1 "Conn_bouton_2" H 3525 2425 50  0000 C CNN
-F 2 "TerminalBlock_Phoenix:TerminalBlock_Phoenix_MPT-0,5-3-2.54_1x03_P2.54mm_Horizontal" H 3175 2400 50  0001 C CNN
-F 3 "~" H 3175 2400 50  0001 C CNN
-	1    3175 2400
-	-1   0    0    1
-$EndComp

Commit message: update
Changed lines of the file:
@@
 Wire Wire Line
 	4525 2200 4525 2300
+Text GLabel 3375 2600 2    50   Output ~ 0
+Vcc_LED
 Text GLabel 3375 2800 2    50   Output ~ 0
-Vcc_LED
-Text GLabel 3375 2600 2    50   Output ~ 0
 GND
 Text GLabel 3375 2100 2    50   Input ~ 0

Commit message: update
Connections:
- net labels added: Bouton_Bas, Bouton_Droite, Bouton_Gauche, Bouton_Haut
- net labels removed: Bouton_1, Bouton_2, Bouton_3, Bouton_4
Changed lines of the file:
@@
 encoding utf-8
 Sheet 1 1
-Title ""
-Date ""
+Title "Boutons de jeu"
+Date "2019-05-09"
 Rev ""
-Comp ""
-Comment1 ""
+Comp "CPNV MCT"
+Comment1 "AKC"
 Comment2 ""
 Comment3 ""
@@
 GND
 Text GLabel 3375 2100 2    50   Input ~ 0
-Bouton_1
+Bouton_Gauche
 Text GLabel 3375 2300 2    50   Input ~ 0
-Bouton_2
+Bouton_Bas
 Text GLabel 3375 2500 2    50   Input ~ 0
-Bouton_3
+Bouton_Droite
 Text GLabel 3375 2700 2    50   Input ~ 0
-Bouton_4
+Bouton_Haut
 $Comp
 L Device:R R1
@@
 Vcc_LED
 Text GLabel 5025 1675 2    50   Output ~ 0
-Bouton_1
+Bouton_Gauche
 Text GLabel 5025 2200 2    50   Output ~ 0
-Bouton_2
+Bouton_Bas
 Text GLabel 5025 2750 2    50   Output ~ 0
-Bouton_3
+Bouton_Droite
 Text GLabel 5025 3275 2    50   Output ~ 0
-Bouton_4
+Bouton_Haut
 $Comp
 L Connector_Generic:Conn_01x08 J1
