File: 07_Schémas/manette_2019_boutons/manette_2019_boutons.kicad_pcb (KiCad board)
At the start: 2 copper layers, 50.8 x 40.6 mm, 14 parts, among them J1 Conn_bouton_1, J2 Conn_bouton_2, SW1 Bouton_1, SW2 Bouton_2, SW3 Bouton_3, SW4 Bouton_4

Commit message: update schema
Changed lines of the file:
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@@
     (pad_to_mask_clearance 0.2)
     (aux_axis_origin 0 0)
-    (visible_elements FFFFFF7F)
+    (visible_elements 7FFFFFFF)
     (pcbplotparams
       (layerselection 0x010fc_ffffffff)
@@
   (segment (start 162.56 95.25) (end 163.83 95.25) (width 1) (layer B.Cu) (net 2))
   (segment (start 163.83 95.25) (end 166.37 92.71) (width 1) (layer B.Cu) (net 2))
-  (segment (start 133.35 87.63) (end 138.43 87.63) (width 0.25) (layer B.Cu) (net 3))
-  (segment (start 138.43 87.63) (end 139.7 88.9) (width 0.25) (layer B.Cu) (net 3))
-  (segment (start 139.7 88.9) (end 139.7 91.44) (width 0.25) (layer B.Cu) (net 3))
-  (segment (start 133.35 97.79) (end 149.86 97.79) (width 0.25) (layer B.Cu) (net 4))
-  (segment (start 149.86 97.79) (end 152.4 100.33) (width 0.25) (layer B.Cu) (net 4))
-  (segment (start 152.4 100.33) (end 152.4 102.87) (width 0.25) (layer B.Cu) (net 4))
-  (segment (start 153.67 80.01) (end 154.94 81.28) (width 0.25) (layer B.Cu) (net 6))
-  (segment (start 152.4 80.01) (end 153.67 80.01) (width 0.25) (layer B.Cu) (net 6))
-  (segment (start 154.94 81.28) (end 154.94 88.9) (width 0.25) (layer B.Cu) (net 6))
-  (segment (start 153.67 91.44) (end 165.1 91.44) (width 0.25) (layer B.Cu) (net 5))
-  (segment (start 153.67 91.44) (end 149.86 95.25) (width 0.25) (layer B.Cu) (net 5))
-  (segment (start 149.86 95.25) (end 133.35 95.25) (width 0.25) (layer B.Cu) (net 5))
-  (segment (start 133.35 92.71) (end 137.16 92.71) (width 0.25) (layer B.Cu) (net 6))
-  (segment (start 137.16 92.71) (end 138.43 93.98) (width 0.25) (layer B.Cu) (net 6))
-  (segment (start 138.43 93.98) (end 149.86 93.98) (width 0.25) (layer B.Cu) (net 6))
-  (segment (start 149.86 93.98) (end 152.4 91.44) (width 0.25) (layer B.Cu) (net 6))
-  (segment (start 152.4 91.44) (end 154.94 88.9) (width 0.25) (layer B.Cu) (net 6))
-  (segment (start 149.86 90.17) (end 149.86 91.44) (width 0.25) (layer B.Cu) (net 7))
-  (segment (start 152.4 87.63) (end 149.86 90.17) (width 0.25) (layer B.Cu) (net 7))
-  (segment (start 152.4 82.55) (end 152.4 87.63) (width 0.25) (layer B.Cu) (net 7))
-  (segment (start 147.32 78.74) (end 148.59 78.74) (width 0.25) (layer B.Cu) (net 7))
-  (segment (start 148.59 78.74) (end 152.4 82.55) (width 0.25) (layer B.Cu) (net 7))
-  (segment (start 166.37 100.33) (end 166.37 101.6) (width 0.25) (layer B.Cu) (net 10))
-  (segment (start 166.37 101.6) (end 165.1 102.87) (width 0.25) (layer B.Cu) (net 10))
-  (segment (start 165.1 102.87) (end 162.56 102.87) (width 0.25) (layer B.Cu) (net 10))
-  (segment (start 162.56 80.01) (end 162.56 76.2) (width 0.25) (layer B.Cu) (net 8))
-  (segment (start 162.56 76.2) (end 161.29 74.93) (width 0.25) (layer B.Cu) (net 8))
-  (segment (start 161.29 74.93) (end 147.32 74.93) (width 0.25) (layer B.Cu) (net 8))
-  (segment (start 166.37 95.25) (end 168.91 95.25) (width 0.25) (layer B.Cu) (net 9))
-  (segment (start 168.91 95.25) (end 172.72 91.44) (width 0.25) (layer B.Cu) (net 9))
-  (segment (start 172.72 91.44) (end 175.26 91.44) (width 0.25) (layer B.Cu) (net 9))
-  (segment (start 166.37 100.33) (end 166.37 99.06) (width 0.25) (layer B.Cu) (net 10))
+  (segment (start 133.35 87.63) (end 138.43 87.63) (width 0.5) (layer B.Cu) (net 3))
+  (segment (start 138.43 87.63) (end 139.7 88.9) (width 0.5) (layer B.Cu) (net 3))
+  (segment (start 139.7 88.9) (end 139.7 91.44) (width 0.5) (layer B.Cu) (net 3))
+  (segment (start 133.35 97.79) (end 149.86 97.79) (width 0.5) (layer B.Cu) (net 4))
+  (segment (start 149.86 97.79) (end 152.4 100.33) (width 0.5) (layer B.Cu) (net 4))
+  (segment (start 152.4 100.33) (end 152.4 102.87) (width 0.5) (layer B.Cu) (net 4))
+  (segment (start 153.67 91.44) (end 165.1 91.44) (width 0.5) (layer B.Cu) (net 5))
+  (segment (start 153.67 91.44) (end 149.86 95.25) (width 0.5) (layer B.Cu) (net 5))
+  (segment (start 149.86 95.25) (end 133.35 95.25) (width 0.5) (layer B.Cu) (net 5))
+  (segment (start 153.67 80.01) (end 154.94 81.28) (width 0.5) (layer B.Cu) (net 6))
+  (segment (start 152.4 80.01) (end 153.67 80.01) (width 0.5) (layer B.Cu) (net 6))
+  (segment (start 154.94 81.28) (end 154.94 88.9) (width 0.5) (layer B.Cu) (net 6))
+  (segment (start 133.35 92.71) (end 137.16 92.71) (width 0.5) (layer B.Cu) (net 6))
+  (segment (start 137.16 92.71) (end 138.43 93.98) (width 0.5) (layer B.Cu) (net 6))
+  (segment (start 138.43 93.98) (end 149.86 93.98) (width 0.5) (layer B.Cu) (net 6))
+  (segment (start 149.86 93.98) (end 152.4 91.44) (width 0.5) (layer B.Cu) (net 6))
+  (segment (start 152.4 91.44) (end 154.94 88.9) (width 0.5) (layer B.Cu) (net 6))
+  (segment (start 149.86 90.17) (end 149.86 91.44) (width 0.5) (layer B.Cu) (net 7))
+  (segment (start 152.4 87.63) (end 149.86 90.17) (width 0.5) (layer B.Cu) (net 7))
+  (segment (start 152.4 82.55) (end 152.4 87.63) (width 0.5) (layer B.Cu) (net 7))
+  (segment (start 147.32 78.74) (end 148.59 78.74) (width 0.5) (layer B.Cu) (net 7))
+  (segment (start 148.59 78.74) (end 152.4 82.55) (width 0.5) (layer B.Cu) (net 7))
+  (segment (start 162.56 80.01) (end 162.56 76.2) (width 0.5) (layer B.Cu) (net 8))
+  (segment (start 162.56 76.2) (end 161.29 74.93) (width 0.5) (layer B.Cu) (net 8))
+  (segment (start 161.29 74.93) (end 147.32 74.93) (width 0.5) (layer B.Cu) (net 8))
+  (segment (start 166.37 95.25) (end 168.91 95.25) (width 0.5) (layer B.Cu) (net 9))
+  (segment (start 168.91 95.25) (end 172.72 91.44) (width 0.5) (layer B.Cu) (net 9))
+  (segment (start 172.72 91.44) (end 175.26 91.44) (width 0.5) (layer B.Cu) (net 9))
+  (segment (start 166.37 100.33) (end 166.37 101.6) (width 0.5) (layer B.Cu) (net 10))
+  (segment (start 166.37 101.6) (end 165.1 102.87) (width 0.5) (layer B.Cu) (net 10))
+  (segment (start 165.1 102.87) (end 162.56 102.87) (width 0.5) (layer B.Cu) (net 10))
+  (segment (start 166.37 100.33) (end 166.37 99.06) (width 0.5) (layer B.Cu) (net 10))
   (zone (net 2) (net_name GND) (layer B.Cu) (hatch edge 0.508)
     (connect_pads (clearance 0.508))

Commit message: update schema
Connections:
- net VCC renamed Vcc_LED

Commit message: update schema
Parts:
- removed J2: Conn_bouton_2, TerminalBlock_Phoenix:TerminalBlock_Phoenix_MPT-0,5-3-2.54_1x03_P2.54mm_Horizontal
- J1: value Conn_bouton_1 -> Conn_bouton; footprint TerminalBlock_Phoenix:TerminalBlock_Phoenix_MPT-0,5-3-2.54_1x03_P2.54mm_Horizontal -> manette_2019:Conn_8; moved to B.Cu
- moved J1 5.14 mm to (132.6, 87.6), turned to 90 degrees
- moved REF** 1.27 mm to (132.1, 73.7)
- moved REF** 1.27 mm to (174.0, 73.7)
Connections:
- J1 pad 2: GND -> Bouton_4
- J1 pad 3: Bouton_1 -> GND
Routing:
- net Vcc_LED: track 80.9 -> 98.0 mm
- net GND: track 101.6 -> 114.2 mm
- net Bouton_4: track 22.6 -> 26.1 mm
- net Bouton_3: track 33.3 -> 36.3 mm
- net Bouton_2: track 34.9 -> 37.1 mm
- net Bouton_1: track 9.42 -> 11.5 mm
- net Net-(R3-Pad2): track 10.5 -> 12.1 mm
- net Net-(R1-Pad2): track 16.6 -> 17.9 mm
- net Net-(R2-Pad2): track 19.6 -> 18.7 mm
Other:
- board size 50.8 x 40.6 mm -> 52.1 x 40.6 mm

Commit message: update
Parts:
- J1: moved to F.Cu
- moved R2 46.2 mm to (176.5, 99.1), turned to 180 degrees
- moved R4 46.2 mm to (137.2, 74.9), turned to 0 degrees
- moved SW2 22.9 mm to (157.5, 99.1)
- moved SW4 22.9 mm to (157.5, 76.2)
- moved J1 1.72 mm to (132.0, 89.2), turned to 270 degrees
Connections:
- J1 pad 1: Vcc_LED -> GND
- J1 pad 3: GND -> Vcc_LED
Routing:
- net GND: track 114.2 -> 100.0 mm
- net Net-(R2-Pad2): track 18.7 -> 6.88 mm
- net Net-(R4-Pad2): track 7.02 -> 17.3 mm
- net Bouton_3: track 36.3 -> 44.8 mm
- net Net-(R1-Pad2): track 17.9 -> 26.1 mm
- net Vcc_LED: track 98.0 -> 90.6 mm
- net Bouton_2: track 37.1 -> 30.8 mm
- net Bouton_1: track 11.5 -> 7.84 mm
- net Net-(R3-Pad2): track 12.1 -> 10.5 mm
- net Bouton_4: track 26.1 -> 25.1 mm

Commit message: update
Connections:
- net Bouton_1 renamed Bouton_Gauche
- net Bouton_2 renamed Bouton_Bas
- net Bouton_3 renamed Bouton_Droite
- net Bouton_4 renamed Bouton_Haut
Other:
- outline, holes or cut-outs redrawn
- board text added: "P1701 Manette Boutons de jeu MCT 2018-2019 AKC"
- board text removed: "P1701 Manette Boutons MCT 2018-2019 AKC"

Commit message: update
Parts:
- removed the REF** at (132.1, 105.4)
- removed the REF** at (174.0, 105.4)
- removed the REF** at (132.1, 73.7)
- added REF**: MountingHole_3.2mm_M3, MountingHole:MountingHole_3.2mm_M3, F.Cu at (137.2, 104.1)
- added REF**: MountingHole_3.2mm_M3, MountingHole:MountingHole_3.2mm_M3, F.Cu at (172.7, 104.1)
- moved J1 16.9 mm to (143.5, 101.6)
- moved REF** 1.27 mm to (172.7, 73.7)
Routing:
- net Bouton_Bas: track 30.8 -> 7.62 mm
- net Bouton_Gauche: track 7.84 -> 27.1 mm
- net Bouton_Droite: track 44.8 -> 26.2 mm
- net Vcc_LED: track 90.3 -> 96.0 mm
- net Bouton_Haut: track 25.1 -> 20.9 mm
- net GND: track 100.0 -> 103.4 mm
- net Net-(R1-Pad2): track 26.1 -> 23.2 mm
Other:
- board size 52.1 x 40.6 mm -> 46.4 x 40.6 mm
