File: 07_Schémas/Manette_2019_boutons_centraux/Manette_2019_PCB_Central.kicad_pcb (KiCad board)
At the start: 2 copper layers, 34.9 x 26 mm, 8 parts, among them J1 Conn_Middle_PCB, SW1 Button_Start, SW2 Button_Select

Commit message: update
Other:
- outline, holes or cut-outs redrawn
- board text added: "P1704 Manette Boutons centraux MCT2018-2019 AKC"
- board text removed: "P1704 Manette PCB Central MCT2018-2019 AKC"
Changed lines of the file:
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@@
   (general
     (thickness 1.6)
-    (drawings 5)
+    (drawings 9)
     (tracks 48)
     (zones 0)
@@
     (pad "" np_thru_hole circle (at 5.21 0.53) (size 1.5 1.5) (drill 1.5) (layers *.Cu *.Mask))
   )
-  (gr_text "P1704 Manette\nPCB Central\nMCT2018-2019\nAKC\n" (at 138.303 123.19) (layer B.Cu)
+  (gr_arc (start 111.379 102.997) (end 111.379 99.822) (angle -90) (layer Edge.Cuts) (width 0.15))
+  (gr_arc (start 111.379 122.682) (end 108.204 122.682) (angle -90) (layer Edge.Cuts) (width 0.15))
+  (gr_arc (start 139.954 122.682) (end 139.954 125.857) (angle -90) (layer Edge.Cuts) (width 0.15))
+  (gr_arc (start 139.954 102.997) (end 143.129 102.997) (angle -90) (layer Edge.Cuts) (width 0.15))
+  (gr_text "P1704 Manette\nBoutons centraux\nMCT2018-2019\nAKC\n" (at 138.303 123.19) (layer B.Cu)
     (effects (font (size 0.6 0.6) (thickness 0.15)) (justify mirror))
   )
-  (gr_line (start 108.204 99.822) (end 108.204 125.857) (layer Edge.Cuts) (width 0.15))
-  (gr_line (start 143.129 99.822) (end 108.204 99.822) (layer Edge.Cuts) (width 0.15))
-  (gr_line (start 143.129 125.857) (end 143.129 99.822) (layer Edge.Cuts) (width 0.15))
-  (gr_line (start 108.204 125.857) (end 143.129 125.857) (layer Edge.Cuts) (width 0.15))
-  (segment (start 131.445 114.173) (end 131.445 111.76) (width 1) (layer B.Cu) (net 1))
-  (segment (start 122.809 123.952) (end 123.444 124.587) (width 1) (layer B.Cu) (net 1))
-  (segment (start 122.809 122.428) (end 122.809 123.952) (width 1) (layer B.Cu) (net 1))
-  (segment (start 123.444 124.587) (end 132.334 124.587) (width 1) (layer B.Cu) (net 1))
-  (segment (start 132.334 124.587) (end 132.969 123.952) (width 1) (layer B.Cu) (net 1))
-  (segment (start 132.969 123.952) (end 132.969 115.697) (width 1) (layer B.Cu) (net 1))
-  (segment (start 132.969 115.697) (end 131.445 114.173) (width 1) (layer B.Cu) (net 1))
+  (gr_line (start 108.204 102.997) (end 108.204 122.682) (layer Edge.Cuts) (width 0.15))
+  (gr_line (start 139.954 99.822) (end 111.379 99.822) (layer Edge.Cuts) (width 0.15))
+  (gr_line (start 143.129 122.682) (end 143.129 102.997) (layer Edge.Cuts) (width 0.15))
+  (gr_line (start 111.379 125.857) (end 139.954 125.857) (layer Edge.Cuts) (width 0.15))
+  (segment (start 131.445 114.173) (end 131.445 111.76) (width 0.5) (layer B.Cu) (net 1))
+  (segment (start 122.809 123.952) (end 123.444 124.587) (width 0.5) (layer B.Cu) (net 1))
+  (segment (start 122.809 122.428) (end 122.809 123.952) (width 0.5) (layer B.Cu) (net 1))
+  (segment (start 123.444 124.587) (end 132.334 124.587) (width 0.5) (layer B.Cu) (net 1))
+  (segment (start 132.334 124.587) (end 132.969 123.952) (width 0.5) (layer B.Cu) (net 1))
+  (segment (start 132.969 123.952) (end 132.969 115.697) (width 0.5) (layer B.Cu) (net 1))
+  (segment (start 132.969 115.697) (end 131.445 114.173) (width 0.5) (layer B.Cu) (net 1))
   (segment (start 110.236 111.76) (end 111.76 111.76) (width 0.5) (layer B.Cu) (net 2))
   (segment (start 118.11 122.428) (end 115.189 119.507) (width 0.5) (layer B.Cu) (net 2))
@@
   (segment (start 119.761 111.76) (end 121.92 111.76) (width 0.5) (layer B.Cu) (net 5))
   (segment (start 115.951 115.57) (end 119.761 111.76) (width 0.5) (layer B.Cu) (net 5))
-  (segment (start 126.619 119.888) (end 126.619 118.237) (width 0.5) (layer B.Cu) (net 6))
-  (segment (start 127.635 117.221) (end 127.635 115.57) (width 0.5) (layer B.Cu) (net 6))
-  (segment (start 126.619 118.237) (end 127.635 117.221) (width 0.5) (layer B.Cu) (net 6))
-  (segment (start 123.825 115.57) (end 127.635 115.57) (width 0.5) (layer B.Cu) (net 6))
+  (segment (start 126.619 119.888) (end 126.619 118.237) (width 1) (layer B.Cu) (net 6))
+  (segment (start 127.635 117.221) (end 127.635 115.57) (width 1) (layer B.Cu) (net 6))
+  (segment (start 126.619 118.237) (end 127.635 117.221) (width 1) (layer B.Cu) (net 6))
+  (segment (start 123.825 115.57) (end 127.635 115.57) (width 1) (layer B.Cu) (net 6))
   (segment (start 121.539 119.888) (end 118.11 119.888) (width 0.5) (layer B.Cu) (net 7))
   (segment (start 118.11 119.888) (end 116.459 118.237) (width 0.5) (layer B.Cu) (net 7))
@@
     (polygon
       (pts
-        (xy 108.204 125.222) (xy 133.477 125.222) (xy 133.35 120.65) (xy 142.875 120.65) (xy 142.875 100.33)
-        (xy 108.077 100.33)
+        (xy 110.109 125.222) (xy 133.604 125.222) (xy 133.604 120.142) (xy 142.494 120.142) (xy 142.494 101.092)
+        (xy 110.109 101.092)
       )
     )

Commit message: update
Connections:
- net Vcc renamed +5V
Changed lines of the file:
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@@
     (visible_elements 7FFFFFFF)
     (pcbplotparams
-      (layerselection 0x010fc_ffffffff)
+      (layerselection 0x01000_ffffffff)
       (usegerberextensions false)
       (usegerberattributes false)
@@
       (outputformat 1)
       (mirror false)
-      (drillshape 1)
+      (drillshape 0)
       (scaleselection 1)
-      (outputdirectory ""))
+      (outputdirectory "boutons_centraux/"))
   )
   (net 0 "")
@@
   (net 4 "Net-(R1-Pad2)")
   (net 5 "Net-(R2-Pad2)")
-  (net 6 Vcc)
-  (net 7 Conn_LED_On)
-  (net 8 "Net-(J1-Pad4)")
-  (net 9 "Net-(J1-Pad5)")
-  (net 10 "Net-(J1-Pad7)")
+  (net 6 Conn_LED_On)
+  (net 7 "Net-(J1-Pad4)")
+  (net 8 "Net-(J1-Pad5)")
+  (net 9 "Net-(J1-Pad7)")
+  (net 10 +5V)
   (net_class Default "Ceci est la Netclass par défaut."
     (clearance 0.2)
@@
     (uvia_dia 0.3)
     (uvia_drill 0.1)
+    (add_net +5V)
     (add_net Conn_LED_On)
     (add_net GND)
@@
     (add_net "Net-(R1-Pad2)")
     (add_net "Net-(R2-Pad2)")
-    (add_net Vcc)
     (add_net button_SELECT)
     (add_net button_START)
@@
       (net 4 "Net-(R1-Pad2)"))
     (pad 1 thru_hole circle (at 0 0) (size 2 2) (drill 0.8) (layers *.Cu *.Mask)
-      (net 6 Vcc))
+      (net 10 +5V))
     (model ${KISYS3DMOD}/Resistor_THT.3dshapes/R_Axial_DIN0207_L6.3mm_D2.5mm_P10.16mm_Horizontal.wrl
       (at (xyz 0 0 0))
@@
     )
     (pad 1 thru_hole circle (at 0 0 180) (size 2 2) (drill 0.8) (layers *.Cu *.Mask)
-      (net 6 Vcc))
+      (net 10 +5V))
     (pad 2 thru_hole oval (at 10.16 0 180) (size 2 2) (drill 0.8) (layers *.Cu *.Mask)
       (net 5 "Net-(R2-Pad2)"))
@@
       (net 5 "Net-(R2-Pad2)"))
     (pad 2 thru_hole circle (at -5.08 -3.81) (size 2 2) (drill 0.8) (layers *.Cu *.Mask)
-      (net 7 Conn_LED_On))
+      (net 6 Conn_LED_On))
     (pad 1 thru_hole circle (at 5.08 -3.81) (size 2 2) (drill 0.8) (layers *.Cu *.Mask)
       (net 3 GND))
@@
       (net 2 button_SELECT))
     (pad 2 thru_hole circle (at -3.81 -1.27) (size 2 2) (drill 0.8) (layers *.Cu *.Mask)
-      (net 7 Conn_LED_On))
+      (net 6 Conn_LED_On))
     (pad 3 thru_hole circle (at -2.54 1.27) (size 2 2) (drill 0.8) (layers *.Cu *.Mask)
       (net 1 button_START))
     (pad 4 thru_hole circle (at -1.27 -1.27) (size 2 2) (drill 0.8) (layers *.Cu *.Mask)
-      (net 8 "Net-(J1-Pad4)"))
+      (net 7 "Net-(J1-Pad4)"))
     (pad 5 thru_hole circle (at 0 1.27) (size 2 2) (drill 0.8) (layers *.Cu *.Mask)
-      (net 9 "Net-(J1-Pad5)"))
+      (net 8 "Net-(J1-Pad5)"))
     (pad 6 thru_hole circle (at 1.27 -1.27) (size 2 2) (drill 0.8) (layers *.Cu *.Mask)
-      (net 6 Vcc))
+      (net 10 +5V))
     (pad 7 thru_hole circle (at 2.54 1.27) (size 2 2) (drill 0.8) (layers *.Cu *.Mask)
-      (net 10 "Net-(J1-Pad7)"))
+      (net 9 "Net-(J1-Pad7)"))
     (pad 8 thru_hole circle (at 3.81 -1.27) (size 2 2) (drill 0.8) (layers *.Cu *.Mask)
       (net 3 GND))
@@
   (segment (start 119.761 111.76) (end 121.92 111.76) (width 0.5) (layer B.Cu) (net 5))
   (segment (start 115.951 115.57) (end 119.761 111.76) (width 0.5) (layer B.Cu) (net 5))
-  (segment (start 126.619 119.888) (end 126.619 118.237) (width 1) (layer B.Cu) (net 6))
-  (segment (start 127.635 117.221) (end 127.635 115.57) (width 1) (layer B.Cu) (net 6))
-  (segment (start 126.619 118.237) (end 127.635 117.221) (width 1) (layer B.Cu) (net 6))
-  (segment (start 123.825 115.57) (end 127.635 115.57) (width 1) (layer B.Cu) (net 6))
-  (segment (start 121.539 119.888) (end 118.11 119.888) (width 0.5) (layer B.Cu) (net 7))
-  (segment (start 118.11 119.888) (end 116.459 118.237) (width 0.5) (layer B.Cu) (net 7))
-  (segment (start 116.459 118.237) (end 112.649 118.237) (width 0.5) (layer B.Cu) (net 7))
-  (segment (start 112.649 118.237) (end 111.379 116.967) (width 0.5) (layer B.Cu) (net 7))
-  (segment (start 111.379 116.967) (end 111.379 115.062) (width 0.5) (layer B.Cu) (net 7))
-  (segment (start 111.379 115.062) (end 114.554 111.887) (width 0.5) (layer B.Cu) (net 7))
-  (segment (start 114.554 111.887) (end 114.554 104.902) (width 0.5) (layer B.Cu) (net 7))
-  (segment (start 113.792 104.14) (end 111.76 104.14) (width 0.5) (layer B.Cu) (net 7))
-  (segment (start 114.554 104.902) (end 113.792 104.14) (width 0.5) (layer B.Cu) (net 7))
+  (segment (start 126.619 119.888) (end 126.619 118.237) (width 1) (layer B.Cu) (net 10))
+  (segment (start 127.635 117.221) (end 127.635 115.57) (width 1) (layer B.Cu) (net 10))
+  (segment (start 126.619 118.237) (end 127.635 117.221) (width 1) (layer B.Cu) (net 10))
+  (segment (start 123.825 115.57) (end 127.635 115.57) (width 1) (layer B.Cu) (net 10))
+  (segment (start 121.539 119.888) (end 118.11 119.888) (width 0.5) (layer B.Cu) (net 6))
+  (segment (start 118.11 119.888) (end 116.459 118.237) (width 0.5) (layer B.Cu) (net 6))
+  (segment (start 116.459 118.237) (end 112.649 118.237) (width 0.5) (layer B.Cu) (net 6))
+  (segment (start 112.649 118.237) (end 111.379 116.967) (width 0.5) (layer B.Cu) (net 6))
+  (segment (start 111.379 116.967) (end 111.379 115.062) (width 0.5) (layer B.Cu) (net 6))
+  (segment (start 111.379 115.062) (end 114.554 111.887) (width 0.5) (layer B.Cu) (net 6))
+  (segment (start 114.554 111.887) (end 114.554 104.902) (width 0.5) (layer B.Cu) (net 6))
+  (segment (start 113.792 104.14) (end 111.76 104.14) (width 0.5) (layer B.Cu) (net 6))
+  (segment (start 114.554 104.902) (end 113.792 104.14) (width 0.5) (layer B.Cu) (net 6))
   (zone (net 3) (net_name GND) (layer B.Cu) (hatch edge 0.508)
     (connect_pads (clearance 0.508))
