File: 07_Schémas/Manette_2019_boutons_centraux/Manette_2019_PCB_Central.sch (KiCad schematic (older format))
At the start: 5 parts, among them J1 Conn_Middle_PCB, SW1 Button_Start, SW2 Button_Select

Commit message: update
Changed lines of the file:
@@
 encoding utf-8
 Sheet 1 1
-Title ""
-Date ""
+Title "Boutons Centraux"
+Date "2019-05-09"
 Rev ""
-Comp ""
-Comment1 ""
+Comp "CPNV MCT"
+Comment1 "AKC"
 Comment2 ""
 Comment3 ""
@@
 	1    0    0    -1
 $EndComp
-Text GLabel 2150 2375 2    50   Output ~ 0
+Text GLabel 2150 2475 2    50   Output ~ 0
 Vcc
 Text GLabel 2150 2775 2    50   Input ~ 0
@@
 NoConn ~ 2150 2675
 NoConn ~ 2150 2575
-NoConn ~ 2150 2475
+NoConn ~ 2150 2375
 $EndSCHEMATC

Commit message: update
Connections:
- net labels added: +5V
- net labels removed: Vcc
Changed lines of the file:
@@
 $EndComp
 Text GLabel 2150 2475 2    50   Output ~ 0
-Vcc
++5V
 Text GLabel 2150 2775 2    50   Input ~ 0
 button_START
@@
 Connection ~ 3725 2400
 Text GLabel 5100 2400 2    50   Input ~ 0
-Vcc
++5V
 $Comp
 L Device:R R2
@@
 Conn_LED_On
 Text GLabel 5100 2975 2    50   Input ~ 0
-Vcc
++5V
 Wire Wire Line
 	3725 2300 4400 2300
